Commit message: protobuf

File: uwrt_arm/uwrt_arm_description/urdf/arm/arm.urdf.xacro (robot description, xacro)
@@ -29,6 +29,6 @@
   <xacro:property name="claw_width"               value="0.05"/>  <!-- m -->
   <!-- Joint Properties -->
-  <xacro:property name="turntable_min_angle"      value="-120.0"/> <!-- deg -->
-  <xacro:property name="turntable_max_angle"      value="120.0"/>  <!-- deg -->
+  <xacro:property name="turntable_min_angle"      value="-360.0"/> <!-- deg -->
+  <xacro:property name="turntable_max_angle"      value="360.0"/>  <!-- deg -->
   <xacro:property name="turntable_max_vel"        value="0.5"/>    <!-- rad/s -->
   <xacro:property name="turntable_max_effort"     value="75"/>
@@ -36,6 +36,6 @@
        to represent an "open" chain version of the closed kinematic chain
        on the real robot -->
-  <xacro:property name="shoulder_min_angle"       value="20.0"/> <!-- deg -->
-  <xacro:property name="shoulder_max_angle"       value="75.0"/> <!-- deg -->
+  <xacro:property name="shoulder_min_angle"       value="-360.0"/> <!-- deg -->
+  <xacro:property name="shoulder_max_angle"       value="360.0"/> <!-- deg -->
   <xacro:property name="shoulder_max_effort"      value="75"/>
   <!-- The max speed specified here should be the worst case scenario
@@ -47,14 +47,19 @@
              this maximum acceleration is the lowest over that range -->
   <xacro:property name="shoulder_max_accel"       value="0.1"/> <!-- rad/s^2 -->
-  <xacro:property name="elbow_min_angle"          value="0.0"/>  <!-- deg -->
-  <xacro:property name="elbow_max_angle"          value="80.0"/> <!-- deg -->
+  <xacro:property name="fixed_shoulder_min_angle"       value="-360.0"/> <!-- deg -->
+  <xacro:property name="fixed_shoulder_max_angle"       value="360.0"/> <!-- deg -->
+  <xacro:property name="fixed_shoulder_max_effort"      value="75"/>
+  <xacro:property name="fixed_shoulder_max_vel"         value="1.0"/> <!-- rad/s -->
+  <xacro:property name="fixed_shoulder_max_accel"       value="0.1"/> <!-- rad/s^2 -->
+  <xacro:property name="elbow_min_angle"          value="-360.0"/>  <!-- deg -->
+  <xacro:property name="elbow_max_angle"          value="360.0"/> <!-- deg -->
   <xacro:property name="elbow_max_vel"            value="1.0"/>  <!-- rad/s -->
   <xacro:property name="elbow_max_effort"         value="75"/>
-  <xacro:property name="wrist_roll_min_angle"     value="-135.0"/> <!-- deg -->
-  <xacro:property name="wrist_roll_max_angle"     value="135.0"/>  <!-- deg -->
+  <xacro:property name="wrist_roll_min_angle"     value="-360.0"/> <!-- deg -->
+  <xacro:property name="wrist_roll_max_angle"     value="360.0"/>  <!-- deg -->
   <xacro:property name="wrist_roll_max_vel"       value="1.0"/>    <!-- rad/s -->
   <xacro:property name="wrist_roll_max_effort"    value="75"/>
-  <xacro:property name="wrist_pitch_min_angle"    value="-75.0"/>  <!-- deg -->
-  <xacro:property name="wrist_pitch_max_angle"    value="75.0"/>   <!-- deg -->
+  <xacro:property name="wrist_pitch_min_angle"    value="-360.0"/>  <!-- deg -->
+  <xacro:property name="wrist_pitch_max_angle"    value="360.0"/>   <!-- deg -->
   <xacro:property name="wrist_pitch_max_vel"      value="1.0"/>    <!-- rad/s -->
   <xacro:property name="wrist_pitch_max_effort"   value="100"/>
@@ -144,9 +149,13 @@
     </link>
     <!-- (JOINT) SHOULDER->BICEP (NOT ACTUATED) -->
-    <joint name="${name}_shoulder_bicep_joint" type="fixed">
+    <joint name="${name}_shoulder_bicep_joint" type="revolute">
       <parent link="${name}_shoulder_revolute_link"/>
       <child  link="${name}_bicep_link"/>
       <origin xyz="0 0 ${shoulder_revolute_link_length}"
               rpy="0 ${(180.0 - 60.3) * M_PI / 180.0} 0"/>
+      <limit lower="${fixed_shoulder_min_angle * M_PI / 180.0}"
+             upper="${fixed_shoulder_max_angle * M_PI / 180.0}"
+             effort="${fixed_shoulder_max_effort}"
+             velocity="${fixed_shoulder_max_vel}"/>
     </joint>
     <!-- (LINK) BICEP -->

Commit message: cleanup for working ik

File: uwrt_arm/uwrt_arm_description/urdf/arm/arm.urdf.xacro (robot description, xacro)
@@ -29,6 +29,6 @@
   <xacro:property name="claw_width"               value="0.05"/>  <!-- m -->
   <!-- Joint Properties -->
-  <xacro:property name="turntable_min_angle"      value="-360.0"/> <!-- deg -->
-  <xacro:property name="turntable_max_angle"      value="360.0"/>  <!-- deg -->
+  <xacro:property name="turntable_min_angle"      value="-120.0"/> <!-- deg -->
+  <xacro:property name="turntable_max_angle"      value="120.0"/>  <!-- deg -->
   <xacro:property name="turntable_max_vel"        value="0.5"/>    <!-- rad/s -->
   <xacro:property name="turntable_max_effort"     value="75"/>
@@ -36,6 +36,6 @@
        to represent an "open" chain version of the closed kinematic chain
        on the real robot -->
-  <xacro:property name="shoulder_min_angle"       value="-360.0"/> <!-- deg -->
-  <xacro:property name="shoulder_max_angle"       value="360.0"/> <!-- deg -->
+  <xacro:property name="shoulder_min_angle"       value="20.0"/> <!-- deg -->
+  <xacro:property name="shoulder_max_angle"       value="75.0"/> <!-- deg -->
   <xacro:property name="shoulder_max_effort"      value="75"/>
   <!-- The max speed specified here should be the worst case scenario
@@ -47,19 +47,14 @@
              this maximum acceleration is the lowest over that range -->
   <xacro:property name="shoulder_max_accel"       value="0.1"/> <!-- rad/s^2 -->
-  <xacro:property name="fixed_shoulder_min_angle"       value="-360.0"/> <!-- deg -->
-  <xacro:property name="fixed_shoulder_max_angle"       value="360.0"/> <!-- deg -->
-  <xacro:property name="fixed_shoulder_max_effort"      value="75"/>
-  <xacro:property name="fixed_shoulder_max_vel"         value="1.0"/> <!-- rad/s -->
-  <xacro:property name="fixed_shoulder_max_accel"       value="0.1"/> <!-- rad/s^2 -->
-  <xacro:property name="elbow_min_angle"          value="-360.0"/>  <!-- deg -->
-  <xacro:property name="elbow_max_angle"          value="360.0"/> <!-- deg -->
+  <xacro:property name="elbow_min_angle"          value="0.0"/>  <!-- deg -->
+  <xacro:property name="elbow_max_angle"          value="80.0"/> <!-- deg -->
   <xacro:property name="elbow_max_vel"            value="1.0"/>  <!-- rad/s -->
   <xacro:property name="elbow_max_effort"         value="75"/>
-  <xacro:property name="wrist_roll_min_angle"     value="-360.0"/> <!-- deg -->
-  <xacro:property name="wrist_roll_max_angle"     value="360.0"/>  <!-- deg -->
+  <xacro:property name="wrist_roll_min_angle"     value="-135.0"/> <!-- deg -->
+  <xacro:property name="wrist_roll_max_angle"     value="135.0"/>  <!-- deg -->
   <xacro:property name="wrist_roll_max_vel"       value="1.0"/>    <!-- rad/s -->
   <xacro:property name="wrist_roll_max_effort"    value="75"/>
-  <xacro:property name="wrist_pitch_min_angle"    value="-360.0"/>  <!-- deg -->
-  <xacro:property name="wrist_pitch_max_angle"    value="360.0"/>   <!-- deg -->
+  <xacro:property name="wrist_pitch_min_angle"    value="-75.0"/>  <!-- deg -->
+  <xacro:property name="wrist_pitch_max_angle"    value="75.0"/>   <!-- deg -->
   <xacro:property name="wrist_pitch_max_vel"      value="1.0"/>    <!-- rad/s -->
   <xacro:property name="wrist_pitch_max_effort"   value="100"/>
@@ -149,13 +144,9 @@
     </link>
     <!-- (JOINT) SHOULDER->BICEP (NOT ACTUATED) -->
-    <joint name="${name}_shoulder_bicep_joint" type="revolute">
+    <joint name="${name}_shoulder_bicep_joint" type="fixed">
       <parent link="${name}_shoulder_revolute_link"/>
       <child  link="${name}_bicep_link"/>
       <origin xyz="0 0 ${shoulder_revolute_link_length}"
               rpy="0 ${(180.0 - 60.3) * M_PI / 180.0} 0"/>
-      <limit lower="${fixed_shoulder_min_angle * M_PI / 180.0}"
-             upper="${fixed_shoulder_max_angle * M_PI / 180.0}"
-             effort="${fixed_shoulder_max_effort}"
-             velocity="${fixed_shoulder_max_vel}"/>
     </joint>
     <!-- (LINK) BICEP -->

Commit message: purge of legacy MoveIt! files

File: uwrt_arm/uwrt_arm_description/urdf/arm/arm.urdf.xacro (robot description, xacro)
@@ -36,5 +36,5 @@
        to represent an "open" chain version of the closed kinematic chain
        on the real robot -->
-  <xacro:property name="shoulder_min_angle"       value="20.0"/> <!-- deg -->
+  <xacro:property name="shoulder_min_angle"       value="-20.0"/> <!-- deg -->
   <xacro:property name="shoulder_max_angle"       value="75.0"/> <!-- deg -->
   <xacro:property name="shoulder_max_effort"      value="75"/>
@@ -228,5 +228,5 @@
       <origin xyz="0 0 ${forearm_length + 0.01}"
               rpy="0 0 0"/>
-      <axis xyz="0 0 1"/>
+      <axis xyz="0 1 0"/>
       <limit lower="${wrist_roll_min_angle * M_PI / 180.0}"
              upper="${wrist_roll_max_angle * M_PI / 180.0}"
@@ -271,5 +271,5 @@
       <origin xyz="0 0 0.01"
               rpy="0 0 0"/>
-      <axis xyz="0 1 0"/>
+      <axis xyz="1 0 0"/>
       <limit lower="${wrist_pitch_min_angle * M_PI / 180.0}"
              upper="${wrist_pitch_max_angle * M_PI / 180.0}"
