Commit message: changed leg joint

File: uwrt_mars_rover_description/urdf/robot.xacro (robot description, xacro)
@@ -64,5 +64,5 @@
     <parent link="base_link"/>
     <child link="rocker_${_suffix}"/>
-    <axis xyz="0.0 1.0 0.0"/>
+    <axis xyz="0.0 ${_side*1.0} 0.0"/>
     <limit lower="${-pi/4}" upper="${pi/4}" effort="1000000" velocity="5"/>
   </joint>

Commit message: Separated urdf files and added mode arg to dynamically load components

File: uwrt_mars_rover_description/urdf/robot.xacro (robot description, xacro)
@@ -1,8 +1,12 @@
 <?xml version="1.0" ?>
 <robot name="uwrt_mars_rover" xmlns:xacro="http://www.ros.org/wiki/xacro">
-<xacro:include filename="$(find uwrt_mars_rover_description)/urdf/robot.gazebo" />
+<gazebo>
+  <plugin filename="libgazebo_ros_control.so" name="gazebo_ros_control"/>
+</gazebo>
+<xacro:include filename="$(find uwrt_mars_rover_description)/urdf/robot_arm.xacro"/>
+<xacro:include filename="$(find uwrt_mars_rover_description)/urdf/robot_chassis.xacro"/>
 <xacro:property name="body_color" value="Gazebo/Cyan"/>
-<xacro:property name="wheel_color" value="Gazebo/Silver"/>
-<xacro:property name="rocker_color" value="Gazebo/Red"/>
+<!-- Get the control_mode from the passed argument. -->
+<xacro:property name="_mode" value="$(arg mode)"/>
 <link name="base_link">
   <inertial>
@@ -32,109 +36,15 @@
   <selfCollide>false</selfCollide>
 </gazebo>
-<xacro:macro name="chassis_to_rocker" params="_suffix _side rotate">
-  <link name="rocker_${_suffix}">
-    <inertial>
-      <origin rpy="0 0 0" xyz="-0.0007397688458582806 -1.0783832098202512e-05 -0.0000060755009578"/>
-      <mass value="373.58767139092913"/>
-      <inertia ixx="15.179593" ixy="-0.000146" ixz="-7.2e-05" iyy="9.170619" iyz="0.000335" izz="9.170464"/>
-    </inertial>
-    <visual>
-      <origin rpy="0 0 0" xyz="0 0.0254 0"/>
-      <geometry>
-        <mesh filename="package://uwrt_mars_rover_description/meshes/rocker.stl" scale="0.0254 0.0254 0.0254"/>
-      </geometry>
-      <material name="Red">
-        <color rgba="1 0 0 1"/>
-      </material>
-    </visual>
-    <collision>
-      <origin rpy="0 0 0" xyz="0 0.0254 0"/>
-      <geometry>
-        <mesh filename="package://uwrt_mars_rover_description/meshes/rocker.stl" scale="0.0254 0.0254 0.0254"/>
-      </geometry>
-    </collision>
-  </link>
-  <gazebo reference="rocker_${_suffix}">
-    <material>${rocker_color}</material>
-    <gravity>true</gravity>
-    <selfCollide>false</selfCollide>
-  </gazebo>
-  <joint name="rocker_${_suffix}_to_chassis" type="revolute">
-    <origin xyz="0 ${_side*0.24289} 0" rpy="0.0 0.0 ${pi*rotate}"/>
-    <parent link="base_link"/>
-    <child link="rocker_${_suffix}"/>
-    <axis xyz="0.0 ${_side*1.0} 0.0"/>
-    <limit lower="${-pi/4}" upper="${pi/4}" effort="1000000" velocity="5"/>
-  </joint>
-  <transmission name="rocker_${_suffix}_trans">
-    <type>transmission_interface/SimpleTransmission</type>
-    <joint name="rocker_${_suffix}_to_chassis">
-      <hardwareInterface>hardware_interface/EffortJointInterface</hardwareInterface>
-    </joint>
-    <actuator name="rocker_${_suffix}_to_chassis_actuator">
-      <hardwareInterface>hardware_interface/EffortJointInterface</hardwareInterface>
-      <mechanicalReduction>1</mechanicalReduction>
-    </actuator>
-  </transmission>
-  <xacro:macro name="rocker_to_wheel" params="suffix side reflect n_side">
-    <link name="wheel_${suffix}_${side}">
-      <inertial>
-        <origin rpy="0 0 0" xyz="-0.0007397688458582806 -1.0783832098202512e-05 -0.0000060755009578"/>
-        <mass value="373.58767139092913"/>
-        <inertia ixx="15.179593" ixy="-0.000146" ixz="-7.2e-05" iyy="9.170619" iyz="0.000335" izz="9.170464"/>
-      </inertial>
-      <visual>
-        <origin rpy="0 0 0" xyz="0 0.09398 0"/>
-        <geometry>
-          <mesh filename="package://uwrt_mars_rover_description/meshes/wheel.stl" scale="0.0254 0.0254 0.0254"/>
-        </geometry>
-        <material name="body_color"/>
-      </visual>
-      <collision>
-        <origin rpy="0 0 0" xyz="0 0.09398 0"/>
-        <geometry>
-          <mesh filename="package://uwrt_mars_rover_description/meshes/wheel.stl" scale="0.0254 0.0254 0.0254"/>
-        </geometry>
-      </collision>
-    </link>
-    <joint name="wheel_${suffix}_${side}_to_rocker" type="continuous">
-      <origin xyz="${n_side*0.381} 0.07414 -0.15636" rpy="0.0 0.0 0.0"/>
-      <parent link="rocker_${suffix}"/>
-      <child link="wheel_${suffix}_${side}"/>
-      <axis xyz="0.0 1.0 0.0"/>
-    </joint>
-    <transmission name="wheel_${suffix}_${side}_trans">
-      <type>transmission_interface/SimpleTransmission</type>
-      <joint name="wheel_${suffix}_${side}_to_rocker">
-        <hardwareInterface>hardware_interface/EffortJointInterface</hardwareInterface>
-      </joint>
-      <actuator name="wheel_${suffix}_${side}_actuator">
-        <hardwareInterface>hardware_interface/EffortJointInterface</hardwareInterface>
-        <mechanicalReduction>1</mechanicalReduction>
-      </actuator>
-    </transmission>
-    <gazebo reference="wheel_${suffix}_${side}">
-      <material>${wheel_color}</material>
-      <mu1>1</mu1>
-      <mu2>1</mu2>
-      <fdir1>1 0 0</fdir1>
-      <minDepth>0.001</minDepth>
-      <maxVel>3.0</maxVel>
-      <gravity>true</gravity>
-      <kp  value="10000000.0" />
-      <kd  value="1.0" />
-      <selfCollide>false</selfCollide>
-    </gazebo>
-  </xacro:macro>
-  <xacro:if value="${_suffix == 'right'}">
-    <xacro:rocker_to_wheel suffix="${_suffix}" side="front" reflect="-1" n_side="-1"/>
-    <xacro:rocker_to_wheel suffix="${_suffix}" side="back" reflect="-1" n_side="1"/>
-  </xacro:if>
-  <xacro:if value="${_suffix == 'left'}">
-    <xacro:rocker_to_wheel suffix="${_suffix}" side="front" reflect="1" n_side="1"/>
-    <xacro:rocker_to_wheel suffix="${_suffix}" side="back" reflect="1" n_side="-1"/>
-  </xacro:if>
-</xacro:macro>
-<xacro:chassis_to_rocker _suffix="left" _side="1" rotate="0"/>
-<xacro:chassis_to_rocker _suffix="right" _side="-1" rotate="1"/>
+<!-- Only the arm or science module will be added to the chassis of the robot for any launch configuration. -->
+<!--  Add the arm to the chassis of the robot. -->
+<xacro:if value="${_mode == 'arm_mission' or _mode == 'arm_only'}">
+  <xacro:arm_to_base base_object="base_link"/>
+</xacro:if>
+<!-- Add the science module to the chassis of the robot. -->
+<xacro:if value="${_mode == 'science_mission' or _mode == 'science_only'}">
+  <!-- TODO: Add the science macro here. -->
+</xacro:if>
+<!-- Add the drivetrain to the chassis. This will be launched in any mode configuration. -->
+<xacro:chassis_to_rocker _suffix="left" _side="1" rotate="0" base_object="base_link"/>
+<xacro:chassis_to_rocker _suffix="right" _side="-1" rotate="1" base_object="base_link"/>
 </robot>

Commit message: Updated inertia for the drivetrain

File: uwrt_mars_rover_description/urdf/robot.xacro (robot description, xacro)
@@ -11,7 +11,7 @@
 <link name="base_link">
   <inertial>
-    <origin rpy="0 0 0" xyz="0.15385713698693046 -0.08778896425180195 -0.2698750000003254"/>
-    <mass value="582.8423997062505"/>
-    <inertia ixx="110.709125" ixy="-0.137662" ixz="-0.012299" iyy="155.023526" iyz="0.0" izz="97.815843"/>
+    <origin rpy="0 0 0" xyz="-0.037262 0.0004 0.05814"/>
+    <mass value="16.69"/>
+    <inertia ixx="1.19749" ixy="0.005489" ixz="0.017255" iyy="1.901358" iyz="0.01166538" izz="1.15907"/>
   </inertial>
   <visual>

File: uwrt_mars_rover_description/urdf/robot_arm.xacro (robot description, xacro)
@@ -2,4 +2,5 @@
 <robot name="uwrt_mars_rover" xmlns:xacro="http://www.ros.org/wiki/xacro">
 <xacro:macro name="arm_to_base" params="base_object">
+<!-- TODO: Correct the inertia and reference frame for the inertia for each link. -->
     <link name="turntable">
         <inertial>
@@ -101,4 +102,7 @@
         <limit lower="${-pi/4}" upper="${pi/4}" effort="10000" velocity="0.5"/>
     </joint>
+    <xacro:macro name="claw_to_arm" params="forearm_link">
+        <!---->
+    </xacro:macro>
 </xacro:macro>
 </robot>

File: uwrt_mars_rover_description/urdf/robot_chassis.xacro (robot description, xacro)
@@ -6,7 +6,7 @@
   <link name="rocker_${_suffix}">
     <inertial>
-      <origin rpy="0 0 0" xyz="-0.0007397688458582806 -1.0783832098202512e-05 -0.0000060755009578"/>
-      <mass value="373.58767139092913"/>
-      <inertia ixx="15.179593" ixy="-0.000146" ixz="-7.2e-05" iyy="9.170619" iyz="0.000335" izz="9.170464"/>
+      <origin rpy="0 0 0" xyz="0.0003 0.02583 0.07381"/>
+      <mass value="4.84"/>
+      <inertia ixx="0.073122" ixy="-0.0001" ixz="0.00015" iyy="0.187572" iyz="0.02183" izz="0.15447"/>
     </inertial>
     <visual>
@@ -51,7 +51,7 @@
     <link name="wheel_${suffix}_${side}">
       <inertial>
-        <origin rpy="0 0 0" xyz="-0.0007397688458582806 -1.0783832098202512e-05 -0.0000060755009578"/>
-        <mass value="373.58767139092913"/>
-        <inertia ixx="15.179593" ixy="-0.000146" ixz="-7.2e-05" iyy="9.170619" iyz="0.000335" izz="9.170464"/>
+        <origin rpy="0 0 0" xyz="0 0 0"/>
+        <mass value="1.32"/>
+        <inertia ixx="0.0137" ixy="0" ixz="0" iyy="0.0191595" iyz="0" izz="0.0137"/>
       </inertial>
       <visual>
