Commit message: Added the main portion of the arm to URDF and fixed TF frames

File: uwrt_mars_rover_description/urdf/robot_arm.xacro (robot description, xacro)
@@ -2,4 +2,103 @@
 <robot name="uwrt_mars_rover" xmlns:xacro="http://www.ros.org/wiki/xacro">
 <xacro:macro name="arm_to_base" params="base_object">
+    <link name="turntable">
+        <inertial>
+            <origin rpy="0 0 0" xyz="-0.0007397688458582806 -1.0783832098202512e-05 -0.0000060755009578"/>
+            <mass value="373.58767139092913"/>
+            <inertia ixx="15.179593" ixy="-0.000146" ixz="-7.2e-05" iyy="9.170619" iyz="0.000335" izz="9.170464"/>
+        </inertial>
+        <visual>
+            <origin rpy="0 0 0" xyz="0 0 0"/>
+            <geometry>
+                <mesh filename="package://uwrt_mars_rover_description/meshes/turntable.stl" scale="0.0254 0.0254 0.0254"/>
+            </geometry>
+            <material name="Red">
+                <color rgba="1 0 0 1"/>
+            </material>
+        </visual>
+        <collision>
+            <origin rpy="0 0 0" xyz="0 0 0"/>
+            <geometry>
+                <mesh filename="package://uwrt_mars_rover_description/meshes/turntable.stl" scale="0.0254 0.0254 0.0254"/>
+            </geometry>
+        </collision>
+    </link>
+    <gazebo reference="turntable">
+        <gravity>true</gravity>
+        <selfCollide>false</selfCollide>
+    </gazebo>
+    <joint name="turntable_to_chassis" type="revolute">
+        <origin xyz="0.2445 0 -0.0222" rpy="0.0 0.0 0.0"/>
+        <parent link="${base_object}"/>
+        <child link="turntable"/>
+        <axis xyz="0.0 0.0 1.0"/>
+        <limit lower="${-pi/4}" upper="${pi/4}" effort="10000" velocity="0.5"/>
+    </joint>
+    <link name="bicep">
+        <inertial>
+            <origin rpy="0 0 0" xyz="-0.0007397688458582806 -1.0783832098202512e-05 -0.0000060755009578"/>
+            <mass value="373.58767139092913"/>
+            <inertia ixx="15.179593" ixy="-0.000146" ixz="-7.2e-05" iyy="9.170619" iyz="0.000335" izz="9.170464"/>
+        </inertial>
+        <visual>
+            <origin rpy="0 0 0" xyz="0 0 -0.0381"/>
+            <geometry>
+                <mesh filename="package://uwrt_mars_rover_description/meshes/bicep.stl" scale="0.0254 0.0254 0.0254"/>
+            </geometry>
+            <material name="Red">
+                <color rgba="1 0 0 1"/>
+            </material>
+        </visual>
+        <collision>
+            <origin rpy="0 0 0" xyz="0 0 -0.0381"/>
+            <geometry>
+                <mesh filename="package://uwrt_mars_rover_description/meshes/bicep.stl" scale="0.0254 0.0254 0.0254"/>
+            </geometry>
+        </collision>
+    </link>
+    <gazebo reference="bicep">
+        <gravity>true</gravity>
+        <selfCollide>false</selfCollide>
+    </gazebo>
+    <joint name="shoulder_joint" type="revolute">
+        <origin xyz="0.015875 0 0.0544576" rpy="0.0 0.0 0.0"/>
+        <parent link="turntable"/>
+        <child link="bicep"/>
+        <axis xyz="0.0 1.0 0.0"/>
+        <limit lower="${-pi/4}" upper="${pi/4}" effort="10000" velocity="0.5"/>
+    </joint>
+    <link name="forearm">
+        <inertial>
+            <origin rpy="0 0 0" xyz="-0.0007397688458582806 -1.0783832098202512e-05 -0.0000060755009578"/>
+            <mass value="373.58767139092913"/>
+            <inertia ixx="15.179593" ixy="-0.000146" ixz="-7.2e-05" iyy="9.170619" iyz="0.000335" izz="9.170464"/>
+        </inertial>
+        <visual>
+            <origin rpy="0 0 0" xyz="0.318874 -0.151281 -0.062292"/>
+            <geometry>
+                <mesh filename="package://uwrt_mars_rover_description/meshes/forearm.stl" scale="0.0254 0.0254 0.0254"/>
+            </geometry>
+            <material name="Red">
+                <color rgba="1 0 0 1"/>
+            </material>
+        </visual>
+        <collision>
+            <origin rpy="0 0 0" xyz="0.318874 -0.151281 -0.062292"/>
+            <geometry>
+                <mesh filename="package://uwrt_mars_rover_description/meshes/forearm.stl" scale="0.0254 0.0254 0.0254"/>
+            </geometry>
+        </collision>
+    </link>
+    <gazebo reference="forearm">
+        <gravity>true</gravity>
+        <selfCollide>false</selfCollide>
+    </gazebo>
+    <joint name="elbow" type="revolute">
+        <origin xyz="0.4019042 -0.0011938 0.0596138" rpy="0.0 0.0 0.0"/>
+        <parent link="bicep"/>
+        <child link="forearm"/>
+        <axis xyz="0.0 1.0 0.0"/>
+        <limit lower="${-pi/4}" upper="${pi/4}" effort="10000" velocity="0.5"/>
+    </joint>
 </xacro:macro>
 </robot>

File: uwrt_mars_rover_description/urdf/robot_chassis.xacro (robot description, xacro)
@@ -11,5 +11,5 @@
     </inertial>
     <visual>
-      <origin rpy="0 0 0" xyz="0 0.0254 0"/>
+      <origin rpy="0 0 ${pi*rotate}" xyz="0 ${_side*0.0254} 0"/>
       <geometry>
         <mesh filename="package://uwrt_mars_rover_description/meshes/rocker.stl" scale="0.0254 0.0254 0.0254"/>
@@ -20,5 +20,5 @@
     </visual>
     <collision>
-      <origin rpy="0 0 0" xyz="0 0.0254 0"/>
+      <origin rpy="0 0 ${pi*rotate}" xyz="0 ${_side*0.0254} 0"/>
       <geometry>
         <mesh filename="package://uwrt_mars_rover_description/meshes/rocker.stl" scale="0.0254 0.0254 0.0254"/>
@@ -32,9 +32,9 @@
   </gazebo>
   <joint name="rocker_${_suffix}_to_chassis" type="revolute">
-    <origin xyz="0 ${_side*0.24289} 0" rpy="0.0 0.0 ${pi*rotate}"/>
+    <origin xyz="0 ${_side*0.24289} 0" rpy="0.0 0.0 0.0"/>
     <parent link="${base_object}"/>
     <child link="rocker_${_suffix}"/>
-    <axis xyz="0.0 ${_side*1.0} 0.0"/>
-    <limit lower="${-pi/4}" upper="${pi/4}" effort="1000000" velocity="5"/>
+    <axis xyz="0.0 1.0 0.0"/>
+    <limit lower="${-pi/4}" upper="${pi/4}" effort="100000" velocity="5"/>
   </joint>
   <transmission name="rocker_${_suffix}_trans">
@@ -56,5 +56,5 @@
       </inertial>
       <visual>
-        <origin rpy="0 0 0" xyz="0 0.09398 0"/>
+        <origin rpy="0 0 0" xyz="0 ${reflect*0.09398} 0"/>
         <geometry>
           <mesh filename="package://uwrt_mars_rover_description/meshes/wheel.stl" scale="0.0254 0.0254 0.0254"/>
@@ -63,5 +63,5 @@
       </visual>
       <collision>
-        <origin rpy="0 0 0" xyz="0 0.09398 0"/>
+        <origin rpy="0 0 0" xyz="0 ${reflect*0.09398} 0"/>
         <geometry>
           <mesh filename="package://uwrt_mars_rover_description/meshes/wheel.stl" scale="0.0254 0.0254 0.0254"/>
@@ -70,5 +70,5 @@
     </link>
     <joint name="wheel_${suffix}_${side}_to_rocker" type="continuous">
-      <origin xyz="${n_side*0.381} 0.07414 -0.15636" rpy="0.0 0.0 0.0"/>
+      <origin xyz="${n_side*0.381} ${reflect*0.07414} -0.15636" rpy="0.0 0.0 0.0"/>
       <parent link="rocker_${suffix}"/>
       <child link="wheel_${suffix}_${side}"/>
@@ -99,6 +99,6 @@
   </xacro:macro>
   <xacro:if value="${_suffix == 'right'}">
-    <xacro:rocker_to_wheel suffix="${_suffix}" side="front" reflect="-1" n_side="-1"/>
-    <xacro:rocker_to_wheel suffix="${_suffix}" side="back" reflect="-1" n_side="1"/>
+    <xacro:rocker_to_wheel suffix="${_suffix}" side="back" reflect="-1" n_side="-1"/>
+    <xacro:rocker_to_wheel suffix="${_suffix}" side="front" reflect="-1" n_side="1"/>
   </xacro:if>
   <xacro:if value="${_suffix == 'left'}">

Commit message: Finalized arm urdf and finalized inertias

File: uwrt_mars_rover_description/urdf/robot_arm.xacro (robot description, xacro)
@@ -1,11 +1,11 @@
 <?xml version="1.0" ?>
 <robot name="uwrt_mars_rover" xmlns:xacro="http://www.ros.org/wiki/xacro">
+<xacro:include filename="$(find uwrt_mars_rover_description)/urdf/robot_claw.xacro"/>
 <xacro:macro name="arm_to_base" params="base_object">
-<!-- TODO: Correct the inertia and reference frame for the inertia for each link. -->
     <link name="turntable">
         <inertial>
-            <origin rpy="0 0 0" xyz="-0.0007397688458582806 -1.0783832098202512e-05 -0.0000060755009578"/>
-            <mass value="373.58767139092913"/>
-            <inertia ixx="15.179593" ixy="-0.000146" ixz="-7.2e-05" iyy="9.170619" iyz="0.000335" izz="9.170464"/>
+            <origin rpy="0 0 0" xyz="-0.00358 0.03422 0.05666"/>
+            <mass value="1.26885"/>
+            <inertia ixx="0.00397" ixy="-0.00035" ixz="0.00084" iyy="0.01033" iyz="-0.00008" izz="0.01305"/>
         </inertial>
         <visual>
@@ -38,7 +38,7 @@
     <link name="bicep">
         <inertial>
-            <origin rpy="0 0 0" xyz="-0.0007397688458582806 -1.0783832098202512e-05 -0.0000060755009578"/>
-            <mass value="373.58767139092913"/>
-            <inertia ixx="15.179593" ixy="-0.000146" ixz="-7.2e-05" iyy="9.170619" iyz="0.000335" izz="9.170464"/>
+            <origin rpy="0 0 0" xyz="0.21949 0.01582 0.16754"/>
+            <mass value="6.480"/>
+            <inertia ixx="0.049355726" ixy="-0.009202176" ixz="-0.033305137" iyy="0.185953394" iyz="-0.000337776" izz="0.156889351"/>
         </inertial>
         <visual>
@@ -71,7 +71,7 @@
     <link name="forearm">
         <inertial>
-            <origin rpy="0 0 0" xyz="-0.0007397688458582806 -1.0783832098202512e-05 -0.0000060755009578"/>
-            <mass value="373.58767139092913"/>
-            <inertia ixx="15.179593" ixy="-0.000146" ixz="-7.2e-05" iyy="9.170619" iyz="0.000335" izz="9.170464"/>
+            <origin rpy="0 0 0" xyz="-0.045 0.15159 0.05923"/>
+            <mass value="1.00758"/>
+            <inertia ixx="0.002383071" ixy="0.0000089677" ixz="-0.000286743" iyy="0.010400499" iyz="-0.000000279" izz="0.012282219"/>
         </inertial>
         <visual>
@@ -102,7 +102,5 @@
         <limit lower="${-pi/4}" upper="${pi/4}" effort="10000" velocity="0.5"/>
     </joint>
-    <xacro:macro name="claw_to_arm" params="forearm_link">
-        <!---->
-    </xacro:macro>
+    <xacro:claw_to_arm forearm_link="forearm"/>
 </xacro:macro>
 </robot>
