Commit message: Refactored xacro and got diff drive controller working

File: uwrt_mars_rover_description/urdf/arm/robot_arm.xacro (robot description, xacro)
@@ -1,5 +1,12 @@
 <?xml version="1.0" ?>
-<robot name="uwrt_mars_rover" xmlns:xacro="http://www.ros.org/wiki/xacro">
-<xacro:include filename="$(find uwrt_mars_rover_description)/urdf/robot_claw.xacro"/>
+<robot name="uwrt_mars_rover_sim" xmlns:xacro="http://www.ros.org/wiki/xacro">
+<xacro:include filename="$(find uwrt_mars_rover_description)/urdf/common.gazebo"/>
+<xacro:include filename="$(find uwrt_mars_rover_description)/urdf/common.trans"/>
+<xacro:include filename="$(find uwrt_mars_rover_description)/urdf/arm/robot_claw.xacro"/>
+<xacro:property name="arm_color" value="Gazebo/Green"/>
+<xacro:property name="bicep_z" value="-0.0381"/>
+<xacro:property name="forearm_x" value="0.318874"/>
+<xacro:property name="forearm_y" value="-0.151281"/>
+<xacro:property name="forearm_z" value="-0.062292"/>
 <xacro:macro name="arm_to_base" params="base_object">
     <link name="turntable">
@@ -21,12 +28,9 @@
             <origin rpy="0 0 0" xyz="0 0 0"/>
             <geometry>
-                <mesh filename="package://uwrt_mars_rover_description/meshes/turntable.stl" scale="0.0254 0.0254 0.0254"/>
+                <mesh filename="package://uwrt_mars_rover_description/meshes/collisions/turntable.dae" scale="0.0254 0.0254 0.0254"/>
             </geometry>
         </collision>
     </link>
-    <gazebo reference="turntable">
-        <gravity>true</gravity>
-        <selfCollide>false</selfCollide>
-    </gazebo>
+    <xacro:basic_gazebo_ref link_name="turntable" color="${arm_color}"/>
     <joint name="turntable_to_chassis" type="revolute">
         <origin xyz="0.2445 0 -0.0222" rpy="0.0 0.0 0.0"/>
@@ -36,12 +40,13 @@
         <limit lower="${-pi/4}" upper="${pi/4}" effort="10000" velocity="0.5"/>
     </joint>
+    <xacro:basic_transmission link_name="turntable" joint_name="turntable_to_chassis" mech_reduction="1"/>
     <link name="bicep">
         <inertial>
-            <origin rpy="0 0 0" xyz="0.21949 0.01582 0.16754"/>
+            <origin rpy="0 0 0" xyz="0.21949 0.01582 ${0.16754 + bicep_z}"/>
             <mass value="6.480"/>
             <inertia ixx="0.049355726" ixy="-0.009202176" ixz="-0.033305137" iyy="0.185953394" iyz="-0.000337776" izz="0.156889351"/>
         </inertial>
         <visual>
-            <origin rpy="0 0 0" xyz="0 0 -0.0381"/>
+            <origin rpy="0 0 0" xyz="0 0 ${bicep_z}"/>
             <geometry>
                 <mesh filename="package://uwrt_mars_rover_description/meshes/bicep.stl" scale="0.0254 0.0254 0.0254"/>
@@ -52,15 +57,12 @@
         </visual>
         <collision>
-            <origin rpy="0 0 0" xyz="0 0 -0.0381"/>
+            <origin rpy="0 0 0" xyz="0 0 ${bicep_z}"/>
             <geometry>
-                <mesh filename="package://uwrt_mars_rover_description/meshes/bicep.stl" scale="0.0254 0.0254 0.0254"/>
+                <mesh filename="package://uwrt_mars_rover_description/meshes/collisions/bicep.dae" scale="0.0254 0.0254 0.0254"/>
             </geometry>
         </collision>
     </link>
-    <gazebo reference="bicep">
-        <gravity>true</gravity>
-        <selfCollide>false</selfCollide>
-    </gazebo>
-    <joint name="shoulder_joint" type="revolute">
+    <xacro:basic_gazebo_ref link_name="bicep" color="${arm_color}"/>
+    <joint name="shoulder" type="revolute">
         <origin xyz="0.015875 0 0.0544576" rpy="0.0 0.0 0.0"/>
         <parent link="turntable"/>
@@ -69,12 +71,13 @@
         <limit lower="${-pi/4}" upper="${pi/4}" effort="10000" velocity="0.5"/>
     </joint>
+    <xacro:basic_transmission link_name="bicep" joint_name="shoulder" mech_reduction="1"/>
     <link name="forearm">
         <inertial>
-            <origin rpy="0 0 0" xyz="-0.045 0.15159 0.05923"/>
+            <origin rpy="0 0 0" xyz="${-0.045 + forearm_x} ${0.15159 + forearm_y} ${0.05923 + forearm_z}"/>
             <mass value="1.00758"/>
             <inertia ixx="0.002383071" ixy="0.0000089677" ixz="-0.000286743" iyy="0.010400499" iyz="-0.000000279" izz="0.012282219"/>
         </inertial>
         <visual>
-            <origin rpy="0 0 0" xyz="0.318874 -0.151281 -0.062292"/>
+            <origin rpy="0 0 0" xyz="${forearm_x} ${forearm_y} ${forearm_z}"/>
             <geometry>
                 <mesh filename="package://uwrt_mars_rover_description/meshes/forearm.stl" scale="0.0254 0.0254 0.0254"/>
@@ -85,14 +88,11 @@
         </visual>
         <collision>
-            <origin rpy="0 0 0" xyz="0.318874 -0.151281 -0.062292"/>
+            <origin rpy="0 0 0" xyz="${forearm_x} ${forearm_y} ${forearm_z}"/>
             <geometry>
-                <mesh filename="package://uwrt_mars_rover_description/meshes/forearm.stl" scale="0.0254 0.0254 0.0254"/>
+                <mesh filename="package://uwrt_mars_rover_description/meshes/collisions/forearm.dae" scale="0.0254 0.0254 0.0254"/>
             </geometry>
         </collision>
     </link>
-    <gazebo reference="forearm">
-        <gravity>true</gravity>
-        <selfCollide>false</selfCollide>
-    </gazebo>
+    <xacro:basic_gazebo_ref link_name="forearm" color="${arm_color}"/>
     <joint name="elbow" type="revolute">
         <origin xyz="0.4019042 -0.0011938 0.0596138" rpy="0.0 0.0 0.0"/>
@@ -102,4 +102,5 @@
         <limit lower="${-pi/4}" upper="${pi/4}" effort="10000" velocity="0.5"/>
     </joint>
+    <xacro:basic_transmission link_name="forearm" joint_name="elbow" mech_reduction="1"/>
     <xacro:claw_to_arm forearm_link="forearm"/>
 </xacro:macro>

File: uwrt_mars_rover_description/urdf/arm/robot_claw.xacro (robot description, xacro)
@@ -1,4 +1,13 @@
 <?xml version="1.0" ?>
-<robot name="uwrt_mars_rover" xmlns:xacro="http://www.ros.org/wiki/xacro">
+<robot name="uwrt_mars_rover_sim" xmlns:xacro="http://www.ros.org/wiki/xacro">
+<xacro:include filename="$(find uwrt_mars_rover_description)/urdf/common.gazebo"/>
+<xacro:include filename="$(find uwrt_mars_rover_description)/urdf/common.trans"/>
+<xacro:include filename="$(find uwrt_mars_rover_description)/urdf/arm/robot_claw.trans"/>
+<xacro:property name="claw_color" value="Gazebo/Blue"/>
+<xacro:property name="claw_static_x" value="0.058"/>
+<xacro:property name="servo_x" value="-0.021"/>
+<xacro:property name="servo_z" value="-0.029"/>
+<xacro:property name="hex_key_x" value="-0.138"/>
+<xacro:property name="hex_key_z" value="-0.005"/>
 <xacro:macro name="claw_to_arm" params="forearm_link">
     <link name="claw_up_down">
@@ -17,15 +26,6 @@
             </material>
         </visual>
-        <collision>
-            <origin rpy="0 0 0" xyz="0 0 0"/>
-            <geometry>
-                <mesh filename="package://uwrt_mars_rover_description/meshes/claw_up_down.stl" scale="0.0254 0.0254 0.0254"/>
-            </geometry>
-        </collision>
     </link>
-    <gazebo reference="claw_up_down">
-        <gravity>true</gravity>
-        <selfCollide>false</selfCollide>
-    </gazebo>
+    <xacro:basic_gazebo_ref link_name="claw_up_down" color="${claw_color}"/>
     <joint name="wrist_up_down" type="revolute">
         <origin xyz="0.355638 0.000418 0" rpy="0.0 0.0 0.0"/>
@@ -35,4 +35,6 @@
         <limit lower="${-pi/4}" upper="${pi/4}" effort="10000" velocity="0.5"/>
     </joint>
+    <!-- TODO: insert custom wrist transmission / modify joints for differential wrist -->
+    <xacro:basic_transmission link_name="claw_up_down" joint_name="wrist_up_down" mech_reduction="1"/>
     <link name="claw_rotate">
         <inertial>
@@ -50,15 +52,6 @@
             </material>
         </visual>
-        <collision>
-            <origin rpy="0 0 0" xyz="0 0 0"/>
-            <geometry>
-                <mesh filename="package://uwrt_mars_rover_description/meshes/claw_rotate.stl" scale="0.0254 0.0254 0.0254"/>
-            </geometry>
-        </collision>
     </link>
-    <gazebo reference="claw_rotate">
-        <gravity>true</gravity>
-        <selfCollide>false</selfCollide>
-    </gazebo>
+    <xacro:basic_gazebo_ref link_name="claw_rotate" color="${claw_color}"/>
     <joint name="wrist_rotate" type="continuous">
         <origin xyz="0 0 0" rpy="0.0 0.0 0.0"/>
@@ -67,12 +60,14 @@
         <axis xyz="1.0 0.0 0.0"/>
     </joint>
+    <!-- TODO: insert custom wrist transmission / modify joints for differential wrist -->
+    <xacro:basic_transmission link_name="claw_rotate" joint_name="wrist_rotate" mech_reduction="1"/>
     <link name="claw_static">
         <inertial>
-            <origin rpy="0 0 0" xyz="-0.02271 -0.00121 0.02018"/>
+            <origin rpy="0 0 0" xyz="${-0.02271 + claw_static_x} -0.00121 0.02018"/>
             <mass value="0.57339"/>
             <inertia ixx="0.0004705087" ixy="-0.0000169291" ixz="-0.0000989304" iyy="0.000579985" iyz="-0.000000533" izz="0.000651862"/>
         </inertial>
         <visual>
-            <origin rpy="0 0 0" xyz="0.058 0 0"/>
+            <origin rpy="0 0 0" xyz="${claw_static_x} 0 0"/>
             <geometry>
                 <mesh filename="package://uwrt_mars_rover_description/meshes/claw_static.stl" scale="0.0254 0.0254 0.0254"/>
@@ -82,15 +77,6 @@
             </material>
         </visual>
-        <collision>
-            <origin rpy="0 0 0" xyz="0.058 0 0"/>
-            <geometry>
-                <mesh filename="package://uwrt_mars_rover_description/meshes/claw_static.stl" scale="0.0254 0.0254 0.0254"/>
-            </geometry>
-        </collision>
     </link>
-    <gazebo reference="claw_static">
-        <gravity>true</gravity>
-        <selfCollide>false</selfCollide>
-    </gazebo>
+    <xacro:basic_gazebo_ref link_name="claw_static" color="${claw_color}"/>
     <joint name="wrist_static" type="fixed">
         <origin xyz="0.0652 0 0" rpy="0.0 0.0 0.0"/>
@@ -100,10 +86,10 @@
     <link name="servo">
         <inertial>
-            <origin rpy="0 0 0" xyz="0.0844 -0.00027 0.00657"/>
+            <origin rpy="0 0 0" xyz="${0.0844 + servo_x} -0.00027 ${0.00657 + servo_z}"/>
             <mass value="0.0535"/>
             <inertia ixx="0.000009626" ixy="0.00000095" ixz="-0.0000095" iyy="0.0000714" iyz="-0.0000003" izz="0.00007375"/>
         </inertial>
         <visual>
-            <origin rpy="0 0 0" xyz="-0.021 0 -0.029"/>
+            <origin rpy="0 0 0" xyz="${servo_x} 0 ${servo_z}"/>
             <geometry>
                 <mesh filename="package://uwrt_mars_rover_description/meshes/servo.stl" scale="0.0254 0.0254 0.0254"/>
@@ -114,5 +100,5 @@
         </visual>
         <collision>
-            <origin rpy="0 0 0" xyz="-0.021 0 -0.029"/>
+            <origin rpy="0 0 0" xyz="${servo_x} 0 ${servo_z}"/>
             <geometry>
                 <mesh filename="package://uwrt_mars_rover_description/meshes/servo.stl" scale="0.0254 0.0254 0.0254"/>
@@ -120,8 +106,5 @@
         </collision>
     </link>
-    <gazebo reference="servo">
-        <gravity>true</gravity>
-        <selfCollide>false</selfCollide>
-    </gazebo>
+    <xacro:basic_gazebo_ref link_name="servo" color="${claw_color}"/>
     <joint name="servo_joint" type="revolute">
         <origin xyz="0.079 0 0.029" rpy="0.0 0.0 0.0"/>
@@ -131,12 +114,13 @@
         <limit lower="${-pi/2}" upper="${pi/2}" effort="10000" velocity="0.5"/>
     </joint>
+    <xacro:basic_transmission link_name="servo" joint_name="servo_joint" mech_reduction="1"/>
     <link name="hex_key">
         <inertial>
-            <origin rpy="0 0 0" xyz="0.105 0 0.004"/>
+            <origin rpy="0 0 0" xyz="${0.105 + hex_key_x} 0 ${0.004 + hex_key_z}"/>
             <mass value="0.0224"/>
             <inertia ixx="0.0000002" ixy="0" ixz="0.0000005" iyy="0.0000117" iyz="0" izz="0.0000117"/>
         </inertial>
         <visual>
-            <origin rpy="0 0 0" xyz="-0.138 0 -0.005"/>
+            <origin rpy="0 0 0" xyz="${hex_key_x} 0 ${hex_key_z}"/>
             <geometry>
                 <mesh filename="package://uwrt_mars_rover_description/meshes/hex_key.stl" scale="0.0254 0.0254 0.0254"/>
@@ -147,5 +131,5 @@
         </visual>
         <collision>
-            <origin rpy="0 0 0" xyz="-0.138 0 -0.005"/>
+            <origin rpy="0 0 0" xyz="${hex_key_x} 0 ${hex_key_z}"/>
             <geometry>
                 <mesh filename="package://uwrt_mars_rover_description/meshes/hex_key.stl" scale="0.0254 0.0254 0.0254"/>
@@ -153,8 +137,5 @@
         </collision>
     </link>
-    <gazebo reference="hex_key">
-        <gravity>true</gravity>
-        <selfCollide>false</selfCollide>
-    </gazebo>
+    <xacro:basic_gazebo_ref link_name="hex_key" color="${claw_color}"/>
     <joint name="hex_joint" type="fixed">
         <origin xyz="0.118 0 -0.024" rpy="0.0 0.0 0.0"/>
@@ -165,5 +146,5 @@
         <link name="gripper_finger_${side}">
             <inertial>
-                <origin rpy="0 0 0" xyz="-0.02271 -0.00121 0.02018"/>
+                <origin rpy="0 0 0" xyz="-0.02271 ${-mirror*0.072-0.00121} 0.02018"/>
                 <mass value="0.0479"/>
                 <inertia ixx="0.0000153325" ixy="-0.000015029" ixz="0" iyy="0.000060103" iyz="-0.000000144" izz="0.000071409"/>
@@ -185,8 +166,5 @@
             </collision>
         </link>
-        <gazebo reference="gripper_finger_${side}">
-            <gravity>true</gravity>
-            <selfCollide>false</selfCollide>
-        </gazebo>
+        <xacro:basic_gazebo_ref link_name="gripper_finger_${side}" color="${claw_color}"/>
         <joint name="gripper_joint_${side}" type="revolute">
             <origin xyz="0.058 ${mirror*0.072} 0" rpy="0.0 0.0 0.0"/>
@@ -196,4 +174,5 @@
             <limit lower="${-pi/4}" upper="${pi/4}" effort="10000" velocity="0.5"/>
         </joint>
+        <xacro:basic_transmission link_name="gripper_finger_${side}" joint_name="gripper_joint_${side}" mech_reduction="1"/>
     </xacro:macro>
     <xacro:gripper_to_claw claw_static_link="claw_static" side="right" mirror="-1"/>

File: uwrt_mars_rover_description/urdf/chassis/robot_chassis.xacro (robot description, xacro)
@@ -1,7 +1,11 @@
 <?xml version="1.0" ?>
-<robot name="uwrt_mars_rover" xmlns:xacro="http://www.ros.org/wiki/xacro">
+<robot name="uwrt_mars_rover_sim" xmlns:xacro="http://www.ros.org/wiki/xacro">
+<xacro:include filename="$(find uwrt_mars_rover_description)/urdf/common.gazebo"/>
+<xacro:include filename="$(find uwrt_mars_rover_description)/urdf/chassis/robot_chassis.gazebo"/>
+<xacro:include filename="$(find uwrt_mars_rover_description)/urdf/chassis/robot_chassis.trans"/>
 <xacro:property name="wheel_color" value="Gazebo/Silver"/>
 <xacro:property name="rocker_color" value="Gazebo/Red"/>
 <xacro:macro name="chassis_to_rocker" params="_suffix _side rotate base_object">
+<!-- TODO: update COM of the rocker components -->
   <link name="rocker_${_suffix}">
     <inertial>
@@ -26,30 +30,17 @@
     </collision>
   </link>
-  <gazebo reference="rocker_${_suffix}">
-    <material>${rocker_color}</material>
-    <gravity>true</gravity>
-    <selfCollide>false</selfCollide>
-  </gazebo>
-  <joint name="rocker_${_suffix}_to_chassis" type="revolute">
+  <xacro:basic_gazebo_ref link_name="rocker_${_suffix}" color="${rocker_color}"/>
+  <!-- TODO: Make this a revolute rocker joint and write the differential bar transmission -->
+  <joint name="rocker_${_suffix}_to_chassis" type="fixed">
     <origin xyz="0 ${_side*0.24289} 0" rpy="0.0 0.0 0.0"/>
     <parent link="${base_object}"/>
     <child link="rocker_${_suffix}"/>
-    <axis xyz="0.0 1.0 0.0"/>
-    <limit lower="${-pi/4}" upper="${pi/4}" effort="100000" velocity="5"/>
+    <!--<axis xyz="0.0 1.0 0.0"/>
+    <limit lower="${-pi/4}" upper="${pi/4}" effort="100000" velocity="5"/>-->
   </joint>
-  <transmission name="rocker_${_suffix}_trans">
-    <type>transmission_interface/SimpleTransmission</type>
-    <joint name="rocker_${_suffix}_to_chassis">
-      <hardwareInterface>hardware_interface/EffortJointInterface</hardwareInterface>
-    </joint>
-    <actuator name="rocker_${_suffix}_to_chassis_actuator">
-      <hardwareInterface>hardware_interface/EffortJointInterface</hardwareInterface>
-      <mechanicalReduction>1</mechanicalReduction>
-    </actuator>
-  </transmission>
   <xacro:macro name="rocker_to_wheel" params="suffix side reflect n_side">
     <link name="wheel_${suffix}_${side}">
       <inertial>
-        <origin rpy="0 0 0" xyz="0 0 0"/>
+        <origin rpy="0 0 0" xyz="0 ${reflect*0.09398} 0"/>
         <mass value="1.32"/>
         <inertia ixx="0.0137" ixy="0" ixz="0" iyy="0.0191595" iyz="0" izz="0.0137"/>
@@ -75,26 +66,6 @@
       <axis xyz="0.0 1.0 0.0"/>
     </joint>
-    <transmission name="wheel_${suffix}_${side}_trans">
-      <type>transmission_interface/SimpleTransmission</type>
-      <joint name="wheel_${suffix}_${side}_to_rocker">
-        <hardwareInterface>hardware_interface/EffortJointInterface</hardwareInterface>
-      </joint>
-      <actuator name="wheel_${suffix}_${side}_actuator">
-        <hardwareInterface>hardware_interface/EffortJointInterface</hardwareInterface>
-        <mechanicalReduction>1</mechanicalReduction>
-      </actuator>
-    </transmission>
-    <gazebo reference="wheel_${suffix}_${side}">
-      <material>${wheel_color}</material>
-      <mu1>1</mu1>
-      <mu2>1</mu2>
-      <fdir1>1 0 0</fdir1>
-      <minDepth>0.001</minDepth>
-      <maxVel>3.0</maxVel>
-      <gravity>true</gravity>
-      <kp  value="10000000.0" />
-      <kd  value="1.0" />
-      <selfCollide>false</selfCollide>
-    </gazebo>
+    <xacro:wheel_gazebo wheel_link="wheel_${suffix}_${side}" color="${wheel_color}"/>
+    <xacro:wheel_transmission link_name="wheel_${suffix}_${side}" joint_name="wheel_${suffix}_${side}_to_rocker" mech_reduction="43.8311688312"/>
   </xacro:macro>
   <xacro:if value="${_suffix == 'right'}">

File: uwrt_mars_rover_description/urdf/robot.xacro (robot description, xacro)
@@ -1,12 +1,14 @@
 <?xml version="1.0" ?>
-<robot name="uwrt_mars_rover" xmlns:xacro="http://www.ros.org/wiki/xacro">
-<gazebo>
-  <plugin filename="libgazebo_ros_control.so" name="gazebo_ros_control"/>
-</gazebo>
-<xacro:include filename="$(find uwrt_mars_rover_description)/urdf/robot_arm.xacro"/>
-<xacro:include filename="$(find uwrt_mars_rover_description)/urdf/robot_chassis.xacro"/>
+<robot name="uwrt_mars_rover_sim" xmlns:xacro="http://www.ros.org/wiki/xacro">
+<xacro:include filename="$(find uwrt_mars_rover_description)/urdf/common.gazebo"/>
+<xacro:include filename="$(find uwrt_mars_rover_description)/urdf/robot.gazebo"/>
+<xacro:include filename="$(find uwrt_mars_rover_description)/urdf/arm/robot_arm.xacro"/>
+<xacro:include filename="$(find uwrt_mars_rover_description)/urdf/chassis/robot_chassis.xacro"/>
 <xacro:property name="body_color" value="Gazebo/Cyan"/>
 <!-- Get the control_mode from the passed argument. -->
 <xacro:property name="_mode" value="$(arg mode)"/>
+<!-- TODO: add transmissions (maybe separate file) to actively controlled joints-->
+<!-- TODO: reconfigure the collisions into simple shapes for reduced CPU load -->
+<!-- TODO: add the counter weight for the chassis / rocker bogey (may need to recalculate inertia / split into two components)-->
 <link name="base_link">
   <inertial>
@@ -31,9 +33,5 @@
   </collision>
 </link>
-<gazebo reference="base_link">
-  <material>${body_color}</material>
-  <gravity>true</gravity>
-  <selfCollide>false</selfCollide>
-</gazebo>
+<xacro:basic_gazebo_ref link_name="base_link" color="${body_color}"/>
 <!-- Only the arm or science module will be added to the chassis of the robot for any launch configuration. -->
 <!--  Add the arm to the chassis of the robot. -->
