Commit message: xacro typo fix

File: uwrt_mars_rover_arm/uwrt_mars_rover_arm_description/uwrt_mars_rover_arm_description/urdf/arm_actuator.xacro (robot description, xacro)
@@ -22,5 +22,5 @@
         <!--  TODO: These are not actually parsed by ros2control yet: https://github.com/ros-controls/ros2_control/issues/32, https://github.com/ros-controls/ros2_control/issues/599 -->
         <plugin>transmission_interface/SimpleTransmission</plugin>
-        <joint name="$arm_{prefix}_joint_actuator" role="arm_joint_{$num}">
+        <joint name="arm_${prefix}_joint_actuator" role="arm_joint_{$num}">
             <!-- <mechanical_reduction>${mechanical_reduction}</mechanical_reduction> -->
         </joint>

Commit message: Rename arm joints

File: uwrt_mars_rover_arm/uwrt_mars_rover_arm_description/uwrt_mars_rover_arm_description/urdf/arm_actuator.xacro (robot description, xacro)
@@ -4,10 +4,10 @@
     <xacro:include filename="$(find uwrt_mars_rover_arm_description)/urdf/values.xacro" />
     <xacro:macro name="arm_actuator" params="prefix num">
-    <ros2_control name="arm_${prefix}_joint_actuator" type="actuator">
+    <ros2_control name="${prefix}_joint" type="actuator">
         <hardware>
         <plugin>uwrt_mars_rover_arm_hw/ArmActuatorInterface</plugin>
         <!-- TODO: CAN interface and Odrive id?-->
         </hardware>
-        <joint name="arm_${prefix}_joint_actuator">
+        <joint name="${prefix}_joint">
         <command_interface name="velocity">
             <param name="min">${-default_limit_vel}</param>
@@ -22,5 +22,5 @@
         <!--  TODO: These are not actually parsed by ros2control yet: https://github.com/ros-controls/ros2_control/issues/32, https://github.com/ros-controls/ros2_control/issues/599 -->
         <plugin>transmission_interface/SimpleTransmission</plugin>
-        <joint name="arm_${prefix}_joint_actuator" role="arm_joint_{$num}">
+        <joint name="${prefix}_joint" role="${prefix}_joint">
             <!-- <mechanical_reduction>${mechanical_reduction}</mechanical_reduction> -->
         </joint>

Commit message: Failing. Working on gazebo_ros2_control bringup.

File: uwrt_mars_rover_arm/uwrt_mars_rover_arm_description/uwrt_mars_rover_arm_description/urdf/arm_actuator.xacro (robot description, xacro)
@@ -4,25 +4,19 @@
     <xacro:include filename="$(find uwrt_mars_rover_arm_description)/urdf/values.xacro" />
     <xacro:macro name="arm_actuator" params="prefix num">
-    <ros2_control name="${prefix}_joint" type="actuator">
-        <hardware>
-        <plugin>uwrt_mars_rover_arm_hw/ArmActuatorInterface</plugin>
-        <!-- CAN interface and Odrive id-->
-        </hardware>
-        <joint name="${prefix}_joint">
-        <command_interface name="velocity">
-            <param name="min">${-default_limit_vel}</param>
-            <param name="max">${default_limit_vel}</param>
-        </command_interface>
-        <state_interface name="position"/>
-        <state_interface name="velocity"/>
-        <state_interface name="iq_current"/>
-        <!-- acceleration, torque -->
-        </joint>
-        <transmission name="transmission_{$num}">
-        <plugin>transmission_interface/SimpleTransmission</plugin>
-        <joint name="${prefix}_joint" role="${prefix}_joint">
-            <!-- <mechanical_reduction>${mechanical_reduction}</mechanical_reduction> -->
-        </joint>
-        </transmission>
+        <ros2_control name="GazeboSystem" type="system">
+            <hardware>
+                <plugin>gazebo_ros2_control/GazeboSystem</plugin>
+                <!-- <plugin>uwrt_mars_rover_arm_hw/ArmActuatorInterface</plugin> -->
+                <!-- CAN interface and Odrive id-->
+            </hardware>
+            <joint name="turntable_joint">
+            <command_interface name="velocity">
+                <param name="min">${-default_limit_vel}</param>
+                <param name="max">${default_limit_vel}</param>
+            </command_interface>
+            <state_interface name="position"/>
+            <state_interface name="velocity"/>
+            <state_interface name="effort"/>
+            </joint>
         </ros2_control>
     </xacro:macro>

File: uwrt_mars_rover_arm/uwrt_mars_rover_arm_description/uwrt_mars_rover_arm_description/urdf/ros2control.xacro (robot description, xacro)
@@ -4,7 +4,15 @@
   <xacro:include filename="$(find uwrt_mars_rover_arm_description)/urdf/arm_actuator.xacro"/>
   <xacro:arm_actuator prefix="turntable" num="0"/>
-  <xacro:arm_actuator prefix="upper_arm" num="0"/>
-  <xacro:arm_actuator prefix="wrist" num="0"/>
-  <xacro:arm_actuator prefix="claw_left" num="0"/>
-  <xacro:arm_actuator prefix="claw_right" num="0"/>
+  <!-- <xacro:arm_actuator prefix="upper_arm" num="0"/> -->
+  <!-- <xacro:arm_actuator prefix="wrist" num="0"/> -->
+  <!-- <xacro:arm_actuator prefix="claw_left" num="0"/> -->
+  <!-- <xacro:arm_actuator prefix="claw_right" num="0"/> -->
+  <gazebo>
+    <plugin filename="libgazebo_ros2_control.so" name="gazebo_ros2_control">
+      <robot_param>robot_description</robot_param>
+      <robot_param_node>robot_state_publisher</robot_param_node>
+      <!-- <robot_sim_type>gazebo_ros2_control/DefaultRobotHWSim</robot_sim_type> -->
+      <parameters>$(find uwrt_mars_rover_arm_description)/config/arm_controllers.yaml</parameters>
+    </plugin>
+  </gazebo>
 </robot>

Commit message: URDF booting in Gazebo ros2_control!

File: uwrt_mars_rover_arm/uwrt_mars_rover_arm_description/uwrt_mars_rover_arm_description/urdf/arm_actuator.xacro (robot description, xacro)
@@ -4,5 +4,5 @@
     <xacro:include filename="$(find uwrt_mars_rover_arm_description)/urdf/values.xacro" />
     <xacro:macro name="arm_actuator" params="prefix num">
-        <ros2_control name="GazeboSystem" type="system">
+        <ros2_control name="arm_robot" type="system">
             <hardware>
                 <plugin>gazebo_ros2_control/GazeboSystem</plugin>
@@ -10,5 +10,5 @@
                 <!-- CAN interface and Odrive id-->
             </hardware>
-            <joint name="turntable_joint">
+            <joint name="${prefix}_joint">
             <command_interface name="velocity">
                 <param name="min">${-default_limit_vel}</param>

File: uwrt_mars_rover_arm/uwrt_mars_rover_arm_description/uwrt_mars_rover_arm_description/urdf/macro.xacro (robot description, xacro)
@@ -12,4 +12,8 @@
                 <xacro:rectangle_visual x="${box_size}" y="${box_size}" z="${box_size}"/>
             </collision>
+            <inertial>
+                <mass value ="${default_mass}"/>
+                <xacro:default_inertia/>
+            </inertial>
         </link>
         <joint name = "turntable_joint" type = "continuous">
@@ -32,4 +36,5 @@
         </link>
         <joint name = "shoulder_joint" type = "revolute">
+            <axis xyz="0 0 1"/>
             <parent link = "turntable"/>
             <child link = "upper_arm"/>
@@ -51,4 +56,5 @@
         </link>
         <joint name = "elbow_joint" type = "revolute">
+            <axis xyz="0 0 1.0"/>
             <parent link = "upper_arm"/>
             <child link = "forearm"/>

File: uwrt_mars_rover_arm/uwrt_mars_rover_arm_description/uwrt_mars_rover_arm_description/urdf/ros2control.xacro (robot description, xacro)
@@ -4,13 +4,13 @@
   <xacro:include filename="$(find uwrt_mars_rover_arm_description)/urdf/arm_actuator.xacro"/>
   <xacro:arm_actuator prefix="turntable" num="0"/>
-  <!-- <xacro:arm_actuator prefix="upper_arm" num="0"/> -->
-  <!-- <xacro:arm_actuator prefix="wrist" num="0"/> -->
-  <!-- <xacro:arm_actuator prefix="claw_left" num="0"/> -->
-  <!-- <xacro:arm_actuator prefix="claw_right" num="0"/> -->
+  <xacro:arm_actuator prefix="upper_arm" num="0"/>
+  <xacro:arm_actuator prefix="wrist" num="0"/>
+  <xacro:arm_actuator prefix="claw_left" num="0"/>
+  <xacro:arm_actuator prefix="claw_right" num="0"/>
   <gazebo>
     <plugin filename="libgazebo_ros2_control.so" name="gazebo_ros2_control">
       <robot_param>robot_description</robot_param>
       <robot_param_node>robot_state_publisher</robot_param_node>
-      <!-- <robot_sim_type>gazebo_ros2_control/DefaultRobotHWSim</robot_sim_type> -->
+      <robot_sim_type>gazebo_ros2_control/DefaultRobotHWSim</robot_sim_type>
       <parameters>$(find uwrt_mars_rover_arm_description)/config/arm_controllers.yaml</parameters>
     </plugin>
