Commit message: name change

File: uwrt_mars_rover_arm/uwrt_mars_rover_arm_description/uwrt_mars_rover_arm_description/urdf/macro.xacro (robot description, xacro)
@@ -6,5 +6,5 @@
         <xacro:read_model_data param_file="${param_file}"/>
         <!-- all links and joints -->
-        <link name = "base_link">
+        <link name = "arm_link">
             <visual>
                 <xacro:rectangle_visual x="${box_size}" y="${box_size}" z="${box_size}"/>

Commit message: .

File: uwrt_mars_rover_arm/uwrt_mars_rover_arm_description/uwrt_mars_rover_arm_description/urdf/macro.xacro (robot description, xacro)
@@ -15,5 +15,5 @@
         </link>
         <joint name = "turntable_joint" type = "continuous">
-            <parent link = "base_link"/>
+            <parent link = "arm_link"/>
             <child link = "turntable"/>
             <origin xyz = "0 0 ${box_size/2 + turntable_length/2}"/>

Commit message: Add joint macros.

File: uwrt_mars_rover_arm/uwrt_mars_rover_arm_description/uwrt_mars_rover_arm_description/urdf/macro.xacro (robot description, xacro)
@@ -154,3 +154,28 @@
         </link>
     </xacro:macro>
+    <xacro:macro name="arm_actuator" params="prefix num">
+    <ros2_control name="arm_${prefix}_joint_actuator" type="actuator">
+      <hardware>
+        <plugin>uwrt_mars_rover_arm_hw/ArmActuatorInterface</plugin>
+        <!-- TODO: CAN interface and Odrive id?-->
+      </hardware>
+      <joint name="arm_${prefix}_joint_actuator">
+        <command_interface name="velocity">
+          <param name="min">${-default_limit_vel}</param>
+          <param name="max">${default_limit_vel}</param>
+        </command_interface>
+        <state_interface name="position"/>
+        <state_interface name="velocity"/>
+        <state_interface name="iq_current"/>
+        <!-- TODO: acceleration, torque? -->
+      </joint>
+      <transmission name="transmission_{$num}">
+        <!--  TODO: These are not actually parsed by ros2control yet: https://github.com/ros-controls/ros2_control/issues/32, https://github.com/ros-controls/ros2_control/issues/599 -->
+        <plugin>transmission_interface/SimpleTransmission</plugin>
+        <joint name="$arm_{prefix}_joint_actuator" role="arm_joint_{$num}">
+          <mechanical_reduction>${mechanical_reduction}</mechanical_reduction>
+        </joint>
+      </transmission>
+    </ros2_control>
+  </xacro:macro>
 </robot>

Commit message: Reformat URDF for easier reading

File: uwrt_mars_rover_arm/uwrt_mars_rover_arm_description/uwrt_mars_rover_arm_description/urdf/macro.xacro (robot description, xacro)
@@ -3,6 +3,5 @@
     <!-- file with common value -->
     <xacro:include filename="$(find uwrt_mars_rover_arm_description)/urdf/values.xacro" />
-    <xacro:macro name="robot" params="param_file">
-        <xacro:read_model_data param_file="${param_file}"/>
+    <xacro:macro name="robot">
         <!-- all links and joints -->
         <link name = "base_link">
@@ -154,28 +153,3 @@
         </link>
     </xacro:macro>
-    <xacro:macro name="arm_actuator" params="prefix num">
-    <ros2_control name="arm_${prefix}_joint_actuator" type="actuator">
-      <hardware>
-        <plugin>uwrt_mars_rover_arm_hw/ArmActuatorInterface</plugin>
-        <!-- TODO: CAN interface and Odrive id?-->
-      </hardware>
-      <joint name="arm_${prefix}_joint_actuator">
-        <command_interface name="velocity">
-          <param name="min">${-default_limit_vel}</param>
-          <param name="max">${default_limit_vel}</param>
-        </command_interface>
-        <state_interface name="position"/>
-        <state_interface name="velocity"/>
-        <state_interface name="iq_current"/>
-        <!-- TODO: acceleration, torque? -->
-      </joint>
-      <transmission name="transmission_{$num}">
-        <!--  TODO: These are not actually parsed by ros2control yet: https://github.com/ros-controls/ros2_control/issues/32, https://github.com/ros-controls/ros2_control/issues/599 -->
-        <plugin>transmission_interface/SimpleTransmission</plugin>
-        <joint name="$arm_{prefix}_joint_actuator" role="arm_joint_{$num}">
-          <mechanical_reduction>${mechanical_reduction}</mechanical_reduction>
-        </joint>
-      </transmission>
-    </ros2_control>
-  </xacro:macro>
 </robot>

File: uwrt_mars_rover_arm/uwrt_mars_rover_arm_description/uwrt_mars_rover_arm_description/urdf/urdf.xacro (robot description, xacro)
@@ -1,6 +1,9 @@
 <?xml version="1.0"?>
 <robot xmlns:xacro="http://wiki.ros.org/xacro" name="arm_robot">
-    <xacro:include filename="$(find uwrt_mars_rover_arm_description)/urdf/macro.xacro"/>
+    <!-- <xacro:include filename="$(find uwrt_mars_rover_arm_description)/urdf/macro.xacro"/> -->
+    <xacro:include filename="$(find uwrt_mars_rover_arm_description)/urdf/arm_actuator.xacro"/>
+    <xacro:include filename="$(find uwrt_mars_rover_arm_description)/urdf/values.xacro"/>
+    <xacro:read_model_data param_file="$(find uwrt_mars_rover_arm_description)/urdf/arm_params.yaml"/>
     <xacro:include filename="$(find uwrt_mars_rover_arm_description)/urdf/ros2control.xacro"/>
-    <xacro:robot param_file="$(find uwrt_mars_rover_arm_description)/urdf/arm_params.yaml"/>
+    <!-- <xacro:robot/> -->
 </robot>

Commit message: Fixed velocity controllers.

File: uwrt_mars_rover_arm/uwrt_mars_rover_arm_description/uwrt_mars_rover_arm_description/urdf/macro.xacro (robot description, xacro)
@@ -4,4 +4,12 @@
     <xacro:include filename="$(find uwrt_mars_rover_arm_description)/urdf/values.xacro" />
     <xacro:macro name="robot">
+        <!--
+            TODO: Use a dummy link to avoid the "base links can't have inertias" error when booting this into Gazebo.
+            <link name="dummy"/>
+            <joint name="dummy_to_base_link=" type="fixed">
+                <parent link="dummy"/>
+                <child link="base_link"/>
+            </joint>
+        -->
         <!-- all links and joints -->
         <link name = "base_link">

File: uwrt_mars_rover_arm/uwrt_mars_rover_arm_description/uwrt_mars_rover_arm_description/urdf/ros2control.xacro (robot description, xacro)
@@ -4,6 +4,8 @@
   <xacro:include filename="$(find uwrt_mars_rover_arm_description)/urdf/arm_actuator.xacro"/>
   <xacro:arm_actuator prefix="turntable" num="0"/>
-  <xacro:arm_actuator prefix="upper_arm" num="0"/>
+  <xacro:arm_actuator prefix="shoulder" num="0"/>
   <xacro:arm_actuator prefix="wrist" num="0"/>
+  <xacro:arm_actuator prefix="roll" num="0"/>
+  <xacro:arm_actuator prefix="elbow" num="0"/>
   <xacro:arm_actuator prefix="claw_left" num="0"/>
   <xacro:arm_actuator prefix="claw_right" num="0"/>
