Commit message: add gazebo launch

File: uwrt_mars_rover_drivetrain/uwrt_mars_rover_drivetrain_description/urdf/drivetrain.macro_BACKUP_4743.xacro (robot description, xacro)
@@ -77,4 +77,5 @@
     </link>
   </xacro:macro>
+<<<<<<< HEAD
   <!-- drivetrain macro only for the simulation stuff -->
   <xacro:macro name="drivetrain_actuator_gazebo" params="prefix suffix">
@@ -92,4 +93,7 @@
     <!-- convert the can_id argument to an xacro property -->
     <xacro:property name="can_id_prop" value="${can_id}"/>
+=======
+  <xacro:macro name="drivetrain_actuator" params="prefix suffix sim_gazebo_classic:=^|false">
+>>>>>>> a49a103... add gazebo launch
     <ros2_control name="${prefix}_${suffix}_wheel_actuator" type="actuator">
       <hardware>
@@ -99,6 +103,11 @@
         <xacro:unless value="${sim_gazebo_classic}">
         <plugin>uwrt_mars_rover_drivetrain_hw/UWRTMarsRoverDrivetrainHWActuatorInterface</plugin>
+<<<<<<< HEAD
         <param name="can_id">${can_id_prop}</param>
         <!-- TODO: CAN interface?-->
+=======
+        <!-- TODO: CAN interface and Odrive id?-->
+        </xacro:unless>
+>>>>>>> a49a103... add gazebo launch
       </hardware>
       <joint name="${prefix}_${suffix}_wheel_joint">

File: uwrt_mars_rover_drivetrain/uwrt_mars_rover_drivetrain_description/urdf/drivetrain.macro_BASE_4743.xacro (robot description, xacro)
@@ -12,10 +12,8 @@
     <xacro:property name="chassis_width" value="${chassis_parameters['width']}" scope="parent"/>
     <xacro:property name="chassis_height" value="${chassis_parameters['height']}" scope="parent"/>
-    <xacro:property name="chassis_mass" value="${chassis_parameters['mass']}" scope="parent"/>
     <!-- wheel parameters -->
     <xacro:property name="wheel_diameter" value="${wheel_parameters['diameter']}" scope="parent"/>
     <xacro:property name="wheel_width" value="${wheel_parameters['width']}" scope="parent"/>
     <xacro:property name="wheel_mass" value="${wheel_parameters['mass']}" scope="parent"/>
-    <xacro:property name="wheel_radius" value="${(wheel_parameters['diameter'])/2}" scope="parent"/>
     <!-- control parameters -->
     <xacro:property name="mechanical_reduction" value="${control_parameters['mechanical_reduction']}" scope="parent"/>
@@ -31,22 +29,4 @@
     </inertial>
   </xacro:macro>
-   <xacro:macro name="chassis_inertia" params="chassis_width:=^ chassis_height:=^ chassis_length:=^ chassis_mass:=^">
-    <inertial>
-      <mass value="${chassis_mass}" />
-      <inertia
-          ixx="${(1/12)*(((chassis_height)*(chassis_height))+((chassis_width)*(chassis_width)))}" ixy="0.0" ixz="0.0"
-          iyy="${(1/12)*(((chassis_height)*(chassis_height))+((chassis_length)*(chassis_length)))}" iyz="0.0"
-          izz="${(1/12)*(((chassis_width)*(chassis_width))+((chassis_length)*(chassis_length)))}"/>
-    </inertial>
-  </xacro:macro>
-  <xacro:macro name="wheel_intertia" params="wheel_radius:=^ wheel_width:=^ wheel_mass:=^">
-    <inertial>
-      <mass value="${wheel_mass}" />
-      <inertia
-          ixx="${(1/12)*(3*((wheel_radius)*(wheel_radius))+((wheel_width)*(wheel_width)))}" ixy="0.0" ixz="0.0"
-          iyy="${(1/12)*(3*((wheel_radius)*(wheel_radius))+((wheel_width)*(wheel_width)))}" iyz="0.0"
-          izz="${(1/2)*((wheel_radius)*(wheel_radius))}"/>
-    </inertial>
-  </xacro:macro>
   <xacro:macro name="identical_visual_collision" params="**identical_blocks">
     <visual>
@@ -57,5 +37,4 @@
     </collision>
   </xacro:macro>
-  <!-- macro for the wheel -->
   <xacro:macro name="wheel" params="prefix suffix parent_link reflect wheel_diameter:=^ wheel_width:=^ wheel_mass:=^ wheelbase_length:=^ x_position" >
     <joint name="${prefix}_${suffix}_wheel_joint" type="continuous">
@@ -74,31 +53,12 @@
         </idential_blocks>
       </xacro:identical_visual_collision>
-      <xacro:wheel_intertia />
+      <xacro:default_inertial mass="${wheel_mass}"/>
     </link>
   </xacro:macro>
-  <!-- drivetrain macro only for the simulation stuff -->
-  <xacro:macro name="drivetrain_actuator_gazebo" params="prefix suffix">
-      <joint name="${prefix}_${suffix}_wheel_joint">
-        <command_interface name="velocity">
-          <param name="min">${-max_speed}</param>
-          <param name="max">${max_speed}</param>
-        </command_interface>
-        <state_interface name="position"/>
-        <state_interface name="velocity"/>
-      </joint>
-  </xacro:macro>
-  <!-- actual hardware -->
-  <xacro:macro name="drivetrain_actuator" params="prefix suffix can_id">
-    <!-- convert the can_id argument to an xacro property -->
-    <xacro:property name="can_id_prop" value="${can_id}"/>
+  <xacro:macro name="drivetrain_actuator" params="prefix suffix">
     <ros2_control name="${prefix}_${suffix}_wheel_actuator" type="actuator">
       <hardware>
-        <xacro:if value="${sim_gazebo_classic}">
-          <plugin>gazebo_ros2_control/GazeboSystem</plugin>
-        </xacro:if>
-        <xacro:unless value="${sim_gazebo_classic}">
         <plugin>uwrt_mars_rover_drivetrain_hw/UWRTMarsRoverDrivetrainHWActuatorInterface</plugin>
-        <param name="can_id">${can_id_prop}</param>
-        <!-- TODO: CAN interface?-->
+        <!-- TODO: CAN interface and Odrive id?-->
       </hardware>
       <joint name="${prefix}_${suffix}_wheel_joint">
@@ -109,14 +69,14 @@
         <state_interface name="position"/>
         <state_interface name="velocity"/>
-        <!-- <state_interface name="iq_current"/> -->
+        <state_interface name="iq_current"/>
         <!-- TODO: acceleration, torque? -->
       </joint>
-      <!-- <transmission name="transmission1"> -->
-         <!-- TODO: These are not actually parsed by ros2control yet: https://github.com/ros-controls/ros2_control/issues/32, https://github.com/ros-controls/ros2_control/issues/599 -->
-        <!-- <plugin>transmission_interface/SimpleTransmission</plugin> -->
-        <!-- <joint name="${prefix}_${suffix}_wheel_joint" role="joint1"> -->
-          <!-- <mechanical_reduction>${mechanical_reduction}</mechanical_reduction> -->
-        <!-- </joint> -->
-      <!-- </transmission> -->
+      <transmission name="transmission1">
+        <!--  TODO: These are not actually parsed by ros2control yet: https://github.com/ros-controls/ros2_control/issues/32, https://github.com/ros-controls/ros2_control/issues/599 -->
+        <plugin>transmission_interface/SimpleTransmission</plugin>
+        <joint name="${prefix}_${suffix}_wheel_joint" role="joint1">
+          <mechanical_reduction>${mechanical_reduction}</mechanical_reduction>
+        </joint>
+      </transmission>
     </ros2_control>
   </xacro:macro>

File: uwrt_mars_rover_drivetrain/uwrt_mars_rover_drivetrain_description/urdf/drivetrain.macro_LOCAL_4743.xacro (robot description, xacro)
@@ -94,8 +94,4 @@
     <ros2_control name="${prefix}_${suffix}_wheel_actuator" type="actuator">
       <hardware>
-        <xacro:if value="${sim_gazebo_classic}">
-          <plugin>gazebo_ros2_control/GazeboSystem</plugin>
-        </xacro:if>
-        <xacro:unless value="${sim_gazebo_classic}">
         <plugin>uwrt_mars_rover_drivetrain_hw/UWRTMarsRoverDrivetrainHWActuatorInterface</plugin>
         <param name="can_id">${can_id_prop}</param>

File: uwrt_mars_rover_drivetrain/uwrt_mars_rover_drivetrain_description/urdf/drivetrain.macro_REMOTE_4743.xacro (robot description, xacro)
@@ -12,10 +12,8 @@
     <xacro:property name="chassis_width" value="${chassis_parameters['width']}" scope="parent"/>
     <xacro:property name="chassis_height" value="${chassis_parameters['height']}" scope="parent"/>
-    <xacro:property name="chassis_mass" value="${chassis_parameters['mass']}" scope="parent"/>
     <!-- wheel parameters -->
     <xacro:property name="wheel_diameter" value="${wheel_parameters['diameter']}" scope="parent"/>
     <xacro:property name="wheel_width" value="${wheel_parameters['width']}" scope="parent"/>
     <xacro:property name="wheel_mass" value="${wheel_parameters['mass']}" scope="parent"/>
-    <xacro:property name="wheel_radius" value="${(wheel_parameters['diameter'])/2}" scope="parent"/>
     <!-- control parameters -->
     <xacro:property name="mechanical_reduction" value="${control_parameters['mechanical_reduction']}" scope="parent"/>
@@ -31,22 +29,4 @@
     </inertial>
   </xacro:macro>
-   <xacro:macro name="chassis_inertia" params="chassis_width:=^ chassis_height:=^ chassis_length:=^ chassis_mass:=^">
-    <inertial>
-      <mass value="${chassis_mass}" />
-      <inertia
-          ixx="${(1/12)*(((chassis_height)*(chassis_height))+((chassis_width)*(chassis_width)))}" ixy="0.0" ixz="0.0"
-          iyy="${(1/12)*(((chassis_height)*(chassis_height))+((chassis_length)*(chassis_length)))}" iyz="0.0"
-          izz="${(1/12)*(((chassis_width)*(chassis_width))+((chassis_length)*(chassis_length)))}"/>
-    </inertial>
-  </xacro:macro>
-  <xacro:macro name="wheel_intertia" params="wheel_radius:=^ wheel_width:=^ wheel_mass:=^">
-    <inertial>
-      <mass value="${wheel_mass}" />
-      <inertia
-          ixx="${(1/12)*(3*((wheel_radius)*(wheel_radius))+((wheel_width)*(wheel_width)))}" ixy="0.0" ixz="0.0"
-          iyy="${(1/12)*(3*((wheel_radius)*(wheel_radius))+((wheel_width)*(wheel_width)))}" iyz="0.0"
-          izz="${(1/2)*((wheel_radius)*(wheel_radius))}"/>
-    </inertial>
-  </xacro:macro>
   <xacro:macro name="identical_visual_collision" params="**identical_blocks">
     <visual>
@@ -57,5 +37,4 @@
     </collision>
   </xacro:macro>
-  <!-- macro for the wheel -->
   <xacro:macro name="wheel" params="prefix suffix parent_link reflect wheel_diameter:=^ wheel_width:=^ wheel_mass:=^ wheelbase_length:=^ x_position" >
     <joint name="${prefix}_${suffix}_wheel_joint" type="continuous">
@@ -74,22 +53,8 @@
         </idential_blocks>
       </xacro:identical_visual_collision>
-      <xacro:wheel_intertia />
+      <xacro:default_inertial mass="${wheel_mass}"/>
     </link>
   </xacro:macro>
-  <!-- drivetrain macro only for the simulation stuff -->
-  <xacro:macro name="drivetrain_actuator_gazebo" params="prefix suffix">
-      <joint name="${prefix}_${suffix}_wheel_joint">
-        <command_interface name="velocity">
-          <param name="min">${-max_speed}</param>
-          <param name="max">${max_speed}</param>
-        </command_interface>
-        <state_interface name="position"/>
-        <state_interface name="velocity"/>
-      </joint>
-  </xacro:macro>
-  <!-- actual hardware -->
-  <xacro:macro name="drivetrain_actuator" params="prefix suffix can_id">
-    <!-- convert the can_id argument to an xacro property -->
-    <xacro:property name="can_id_prop" value="${can_id}"/>
+  <xacro:macro name="drivetrain_actuator" params="prefix suffix sim_gazebo_classic:=^|false">
     <ros2_control name="${prefix}_${suffix}_wheel_actuator" type="actuator">
       <hardware>
@@ -99,6 +64,6 @@
         <xacro:unless value="${sim_gazebo_classic}">
         <plugin>uwrt_mars_rover_drivetrain_hw/UWRTMarsRoverDrivetrainHWActuatorInterface</plugin>
-        <param name="can_id">${can_id_prop}</param>
-        <!-- TODO: CAN interface?-->
+        <!-- TODO: CAN interface and Odrive id?-->
+        </xacro:unless>
       </hardware>
       <joint name="${prefix}_${suffix}_wheel_joint">
@@ -109,14 +74,14 @@
         <state_interface name="position"/>
         <state_interface name="velocity"/>
-        <!-- <state_interface name="iq_current"/> -->
+        <state_interface name="iq_current"/>
         <!-- TODO: acceleration, torque? -->
       </joint>
-      <!-- <transmission name="transmission1"> -->
-         <!-- TODO: These are not actually parsed by ros2control yet: https://github.com/ros-controls/ros2_control/issues/32, https://github.com/ros-controls/ros2_control/issues/599 -->
-        <!-- <plugin>transmission_interface/SimpleTransmission</plugin> -->
-        <!-- <joint name="${prefix}_${suffix}_wheel_joint" role="joint1"> -->
-          <!-- <mechanical_reduction>${mechanical_reduction}</mechanical_reduction> -->
-        <!-- </joint> -->
-      <!-- </transmission> -->
+      <transmission name="transmission1">
+        <!--  TODO: These are not actually parsed by ros2control yet: https://github.com/ros-controls/ros2_control/issues/32, https://github.com/ros-controls/ros2_control/issues/599 -->
+        <plugin>transmission_interface/SimpleTransmission</plugin>
+        <joint name="${prefix}_${suffix}_wheel_joint" role="joint1">
+          <mechanical_reduction>${mechanical_reduction}</mechanical_reduction>
+        </joint>
+      </transmission>
     </ros2_control>
   </xacro:macro>

File: uwrt_mars_rover_drivetrain/uwrt_mars_rover_drivetrain_description/urdf/drivetrain.ros2control.xacro (robot description, xacro)
@@ -1,4 +1,5 @@
 <?xml version="1.0"?>
 <robot xmlns:xacro="http://www.ros.org/wiki/xacro">
+  <xacro:arg name="sim_gazebo_classic" default="true" />
   <!-- import macros file -->
   <xacro:include filename="$(find uwrt_mars_rover_drivetrain_description)/urdf/drivetrain.macro.xacro"/>
