Commit message: we got movement!

File: uwrt_mars_rover_drivetrain/uwrt_mars_rover_drivetrain_description/urdf/drivetrain.ros2controlgazebo.xacro (robot description, xacro)
@@ -3,19 +3,24 @@
   <!-- import macros file -->
   <xacro:include filename="$(find uwrt_mars_rover_drivetrain_description)/urdf/drivetrain.macro.xacro"/>
-  <ros2_control name="gazebo_wheel_actuator" type="system">
-    <hardware>
-        <plugin>gazebo_ros2_control/GazeboSystem</plugin>
-    </hardware>
-    <xacro:drivetrain_actuator_gazebo  prefix="right" suffix="front" />
-    <xacro:drivetrain_actuator_gazebo  prefix="right" suffix="middle" />
-    <xacro:drivetrain_actuator_gazebo  prefix="right" suffix="back" />
-    <xacro:drivetrain_actuator_gazebo  prefix="left" suffix="front" />
-    <xacro:drivetrain_actuator_gazebo  prefix="left" suffix="middle" />
-    <xacro:drivetrain_actuator_gazebo  prefix="left" suffix="back" />
-    <gazebo>
-        <plugin filename="libgazebo_ros2_control.so" name="gazebo_ros2_control">
-          <parameters>$(find uwrt_mars_rover_drivetrain_hw)/config/drivetrain_controllers.yaml</parameters>
-        </plugin>
-    </gazebo>
-  </ros2_control>
+  <xacro:macro name="uwrt_drivetrain_ros2_controls">
+    <ros2_control name="gazebo_wheel_actuator" type="system">
+      <hardware>
+          <plugin>gazebo_ros2_control/GazeboSystem</plugin>
+      </hardware>
+      <xacro:drivetrain_actuator_gazebo  prefix="right" suffix="front" />
+      <xacro:drivetrain_actuator_gazebo  prefix="right" suffix="middle" />
+      <xacro:drivetrain_actuator_gazebo  prefix="right" suffix="back" />
+      <xacro:drivetrain_actuator_gazebo  prefix="left" suffix="front" />
+      <xacro:drivetrain_actuator_gazebo  prefix="left" suffix="middle" />
+      <xacro:drivetrain_actuator_gazebo  prefix="left" suffix="back" />
+      <!--  -->
+   </ros2_control>
+      <!-- controller manager -->
+      <gazebo>
+          <plugin filename="libgazebo_ros2_control.so" name="gazebo_ros2_control">
+            <parameters>$(find uwrt_mars_rover_drivetrain_hw)/config/drivetrain_controllers.yaml</parameters>
+            <robot_param_node>/robot_state_publisher </robot_param_node>
+          </plugin>
+      </gazebo>
+  </xacro:macro>
 </robot>

File: uwrt_mars_rover_drivetrain/uwrt_mars_rover_drivetrain_description/urdf/drivetrain.urdf.xacro (robot description, xacro)
@@ -9,18 +9,13 @@
   <!-- calculate parameters based on model data -->
   <xacro:property name="wheelbase_length" value="${chassis_width + wheel_width}"/>
+    <!-- include ros2 control for sim -->
+  <xacro:if value="$(arg sim)">
+      <xacro:include filename="$(find uwrt_mars_rover_drivetrain_description)/urdf/drivetrain.ros2controlgazebo.xacro"/>
+  </xacro:if>
   <!-- include ros2control description for regular -->
   <xacro:unless value="$(arg sim)">
       <xacro:include filename="$(find uwrt_mars_rover_drivetrain_description)/urdf/drivetrain.ros2control.xacro"/>
   </xacro:unless>
-  <!-- include ros2 control for sim -->
-  <xacro:if value="$(arg sim)">
-      <xacro:include filename="$(find uwrt_mars_rover_drivetrain_description)/urdf/drivetrain.ros2controlgazebo.xacro"/>
-  </xacro:if>
   <link name="base_link"/>
-  <joint name="base_link_to_chassis" type="fixed">
-    <parent link="base_link"/>
-    <child link="chassis"/>
-    <origin xyz="0 0 ${wheel_diameter/2}" rpy="0 0 0"/>
-  </joint>
   <link name="chassis">
     <xacro:identical_visual_collision>
@@ -33,10 +28,16 @@
     <xacro:chassis_inertia/>
   </link>
-    <!-- wheels -->
-    <xacro:wheel prefix="right" suffix="front" parent_link="chassis" reflect="-1" x_position="${chassis_length/2}"/>
-    <xacro:wheel prefix="right" suffix="middle" parent_link="chassis" reflect="-1" x_position="0"/>
-    <xacro:wheel prefix="right" suffix="back" parent_link="chassis" reflect="-1" x_position="${-chassis_length/2}"/>
-    <xacro:wheel prefix="left" suffix="front" parent_link="chassis" reflect="1" x_position="${chassis_length/2}"/>
-    <xacro:wheel prefix="left" suffix="middle" parent_link="chassis" reflect="1" x_position="0"/>
-    <xacro:wheel prefix="left" suffix="back" parent_link="chassis" reflect="1" x_position="${-chassis_length/2}"/>
+  <joint name="base_link_to_chassis" type="fixed">
+    <parent link="base_link"/>
+    <child link="chassis"/>
+    <origin xyz="0 0 ${wheel_diameter/2}" rpy="0 0 0"/>
+  </joint>
+  <!-- wheels -->
+  <xacro:wheel prefix="right" suffix="front" parent_link="chassis" reflect="-1" x_position="${chassis_length/2}"/>
+  <xacro:wheel prefix="right" suffix="middle" parent_link="chassis" reflect="-1" x_position="0"/>
+  <xacro:wheel prefix="right" suffix="back" parent_link="chassis" reflect="-1" x_position="${-chassis_length/2}"/>
+  <xacro:wheel prefix="left" suffix="front" parent_link="chassis" reflect="1" x_position="${chassis_length/2}"/>
+  <xacro:wheel prefix="left" suffix="middle" parent_link="chassis" reflect="1" x_position="0"/>
+  <xacro:wheel prefix="left" suffix="back" parent_link="chassis" reflect="1" x_position="${-chassis_length/2}"/>
+  <xacro:uwrt_drivetrain_ros2_controls/>
 </robot>
