Commit message: add macros to simulate sensors

File: uwrt_mars_rover_drivetrain/uwrt_mars_rover_drivetrain_description/urdf/drivetrain.urdf.xacro (robot description, xacro)
@@ -3,7 +3,9 @@
   <!-- import macros file -->
   <xacro:include filename="$(find uwrt_mars_rover_drivetrain_description)/urdf/drivetrain.macro.xacro"/>
+  <xacro:include filename="$(find uwrt_mars_rover_drivetrain_description)/urdf/sensors.macro.xacro"/>
   <!-- load model data from yamls -->
   <xacro:load_model_data
       physical_parameters_file="$(find uwrt_mars_rover_drivetrain_description)/config/physical_parameters.yaml"/>
+  <xacro:property name="sensor_paramater_file" value="$(find uwrt_mars_rover_drivetrain_description)/config/sensor_parameters.yaml"/>
   <!-- calculate parameters based on model data -->
   <xacro:property name="wheelbase_length" value="${chassis_width + wheel_width}"/>
@@ -33,3 +35,9 @@
   <xacro:wheel prefix="left" suffix="middle" parent_link="chassis" reflect="1" x_position="0"/>
   <xacro:wheel prefix="left" suffix="back" parent_link="chassis" reflect="1" x_position="${-chassis_length/2}"/>
+  <!-- sensors -->
+  <xacro:property name="sensors_parameters" value="${load_yaml(sensor_paramater_file)}"/>
+  <xacro:generate_sensor_frame sensor_params="${sensors_parameters['depth_camera']['camera1']}" name="camera1"/>
+  <xacro:default_depth_camera_frame camera_link_name="camera1"/>
+  <xacro:generate_sensor_frame sensor_params="${sensors_parameters['lidar']['lidar1']}"         name="lidar1"/>
+  <xacro:default_lidar_frame lidar_link_name="lidar1"/>
 </robot>

Commit message: add more params to yaml

File: uwrt_mars_rover_drivetrain/uwrt_mars_rover_drivetrain_description/urdf/drivetrain.urdf.xacro (robot description, xacro)
@@ -38,6 +38,8 @@
   <xacro:property name="sensors_parameters" value="${load_yaml(sensor_paramater_file)}"/>
   <xacro:generate_sensor_frame sensor_params="${sensors_parameters['depth_camera']['camera1']}" name="camera1"/>
-  <xacro:default_depth_camera_frame camera_link_name="camera1"/>
-  <xacro:generate_sensor_frame sensor_params="${sensors_parameters['lidar']['lidar1']}"         name="lidar1"/>
-  <xacro:default_lidar_frame lidar_link_name="lidar1"/>
+  <xacro:default_depth_camera_frame camera_link_name="camera1" camera_props="${sensors_parameters['depth_camera']['camera1']['camera_properties']}"/>
+  <xacro:generate_sensor_frame sensor_params="${sensors_parameters['depth_camera']['camera2']}" name="camera2"/>
+  <xacro:default_depth_camera_frame camera_link_name="camera2" camera_props="${sensors_parameters['depth_camera']['camera2']['camera_properties']}"/>
+  <!-- <xacro:generate_sensor_frame sensor_params="${sensors_parameters['lidar']['lidar1']}"         name="lidar1"/>
+  <xacro:default_lidar_frame lidar_link_name="lidar1" lidar_props="${sensors_parameters['lidar']['lidar1']['lidar_properties']}"/> -->
 </robot>

File: uwrt_mars_rover_drivetrain/uwrt_mars_rover_drivetrain_description/urdf/sensors.macro.xacro (robot description, xacro)
@@ -24,5 +24,5 @@
     </joint>
   </xacro:macro>
-  <xacro:macro name="default_depth_camera_frame" params="camera_link_name">
+  <xacro:macro name="default_depth_camera_frame" params="camera_link_name camera_props">
     <gazebo reference="${camera_link_name}">
       <sensor name="${camera_link_name}_sensor" type="depth">
@@ -30,22 +30,22 @@
         <update_rate>30.0</update_rate>
         <camera name="camera">
-          <horizontal_fov>1.047198</horizontal_fov>
+          <horizontal_fov>${camera_props['horizontal_fov']}</horizontal_fov>
           <image>
-            <width>640</width>
-            <height>480</height>
-            <format>R8G8B8</format>
+            <width>${camera_props['image']['width']}</width>
+            <height>${camera_props['image']['height']}</height>
+            <format>${camera_props['image']['format']}</format>
           </image>
           <clip>
-            <near>0.05</near>
-            <far>3</far>
+            <near>${camera_props['clip']['near']}</near>
+            <far>${camera_props['clip']['far']}</far>
           </clip>
         </camera>
         <plugin name="depth_camera_controller" filename="libgazebo_ros_camera.so">
           <cameraName>${camera_link_name}</cameraName>
-          <imageTopicName>ir/image_raw</imageTopicName>
-          <cameraInfoTopicName>ir/camera_info</cameraInfoTopicName>
-          <depthImageTopicName>depth/image_raw</depthImageTopicName>
-          <depthImageCameraInfoTopicName>depth/camera_info</depthImageCameraInfoTopicName>
-          <pointCloudTopicName>depth/points</pointCloudTopicName>
+          <imageTopicName>${camera_link_name}_ir/image_raw</imageTopicName>
+          <cameraInfoTopicName>${camera_link_name}_ir/camera_info</cameraInfoTopicName>
+          <depthImageTopicName>${camera_link_name}_depth/image_raw</depthImageTopicName>
+          <depthImageCameraInfoTopicName>${camera_link_name}_depth/camera_info</depthImageCameraInfoTopicName>
+          <pointCloudTopicName>${camera_link_name}_depth/points</pointCloudTopicName>
           <frameName>${camera_link_name}_optical_frame</frameName>
           <baseline>0.2</baseline>
@@ -69,23 +69,23 @@
     </gazebo>
   </xacro:macro>
-  <xacro:macro name="default_lidar_frame" params="lidar_link_name">
+  <xacro:macro name="default_lidar_frame" params="lidar_link_name lidar_props">
     <gazebo reference="${lidar_link_name}">
     <sensor name="${lidar_link_name}_sensor" type="ray">
       <always_on>true</always_on>
       <visualize>true</visualize>
-      <update_rate>5</update_rate>
+      <update_rate>${lidar_props['update_rate']}</update_rate>
       <ray>
         <scan>
           <horizontal>
-            <samples>360</samples>
-            <resolution>1.000000</resolution>
-            <min_angle>0.000000</min_angle>
-            <max_angle>6.280000</max_angle>
+            <samples>${lidar_props['scan']['samples']}</samples>
+            <resolution>${lidar_props['scan']['resolution']}</resolution>
+            <min_angle>${lidar_props['scan']['min_angle']}</min_angle>
+            <max_angle>${lidar_props['scan']['max_angle']}</max_angle>
           </horizontal>
         </scan>
         <range>
-          <min>0.120000</min>
-          <max>3.5</max>
-          <resolution>0.015000</resolution>
+          <min>${lidar_props['range']['min']}</min>
+          <max>${lidar_props['range']['max']}</max>
+          <resolution>${lidar_props['range']['resolution']}</resolution>
         </range>
         <noise>
@@ -96,7 +96,4 @@
       </ray>
       <plugin name="lidar_controller" filename="libgazebo_ros_ray_sensor.so">
-        <ros>
-          <remapping>~/out:=${lidar_link_name}_sensor/scan</remapping>
-        </ros>
         <output_type>sensor_msgs/LaserScan</output_type>
         <frame_name>${lidar_link_name}</frame_name>

Commit message: PERCEPTION: Setting up sensors (#252)
* add macros to simulate sensors

* add more params to yaml

* add lidar at front

File: uwrt_mars_rover_drivetrain/uwrt_mars_rover_drivetrain_description/urdf/drivetrain.urdf.xacro (robot description, xacro)
@@ -3,7 +3,9 @@
   <!-- import macros file -->
   <xacro:include filename="$(find uwrt_mars_rover_drivetrain_description)/urdf/drivetrain.macro.xacro"/>
+  <xacro:include filename="$(find uwrt_mars_rover_drivetrain_description)/urdf/sensors.macro.xacro"/>
   <!-- load model data from yamls -->
   <xacro:load_model_data
       physical_parameters_file="$(find uwrt_mars_rover_drivetrain_description)/config/physical_parameters.yaml"/>
+  <xacro:property name="sensor_paramater_file" value="$(find uwrt_mars_rover_drivetrain_description)/config/sensor_parameters.yaml"/>
   <!-- calculate parameters based on model data -->
   <xacro:property name="wheelbase_length" value="${chassis_width + wheel_width}"/>
@@ -33,3 +35,11 @@
   <xacro:wheel prefix="left" suffix="middle" parent_link="chassis" reflect="1" x_position="0"/>
   <xacro:wheel prefix="left" suffix="back" parent_link="chassis" reflect="1" x_position="${-chassis_length/2}"/>
+  <!-- sensors -->
+  <xacro:property name="sensors_parameters" value="${load_yaml(sensor_paramater_file)}"/>
+  <xacro:generate_sensor_frame sensor_params="${sensors_parameters['depth_camera']['camera1']}" name="camera1"/>
+  <xacro:default_depth_camera_frame camera_link_name="camera1" camera_props="${sensors_parameters['depth_camera']['camera1']['camera_properties']}"/>
+  <xacro:generate_sensor_frame sensor_params="${sensors_parameters['depth_camera']['camera2']}" name="camera2"/>
+  <xacro:default_depth_camera_frame camera_link_name="camera2" camera_props="${sensors_parameters['depth_camera']['camera2']['camera_properties']}"/>
+  <xacro:generate_sensor_frame sensor_params="${sensors_parameters['lidar']['lidar1']}"         name="lidar1"/>
+  <xacro:default_lidar_frame lidar_link_name="lidar1" lidar_props="${sensors_parameters['lidar']['lidar1']['lidar_properties']}"/>
 </robot>

Commit message: costmap layers

File: uwrt_mars_rover_drivetrain/uwrt_mars_rover_drivetrain_description/urdf/drivetrain.urdf.xacro (robot description, xacro)
@@ -39,6 +39,6 @@
   <xacro:generate_sensor_frame sensor_params="${sensors_parameters['depth_camera']['camera1']}" name="camera1"/>
   <xacro:default_depth_camera_frame camera_link_name="camera1" camera_props="${sensors_parameters['depth_camera']['camera1']['camera_properties']}"/>
-  <xacro:generate_sensor_frame sensor_params="${sensors_parameters['depth_camera']['camera2']}" name="camera2"/>
-  <xacro:default_depth_camera_frame camera_link_name="camera2" camera_props="${sensors_parameters['depth_camera']['camera2']['camera_properties']}"/>
+  <!-- <xacro:generate_sensor_frame sensor_params="${sensors_parameters['depth_camera']['camera2']}" name="camera2"/>
+  <xacro:default_depth_camera_frame camera_link_name="camera2" camera_props="${sensors_parameters['depth_camera']['camera2']['camera_properties']}"/> -->
   <xacro:generate_sensor_frame sensor_params="${sensors_parameters['lidar']['lidar1']}"         name="lidar1"/>
   <xacro:default_lidar_frame lidar_link_name="lidar1" lidar_props="${sensors_parameters['lidar']['lidar1']['lidar_properties']}"/>

File: uwrt_mars_rover_drivetrain/uwrt_mars_rover_drivetrain_description/urdf/sensors.macro.xacro (robot description, xacro)
@@ -25,4 +25,14 @@
   </xacro:macro>
   <xacro:macro name="default_depth_camera_frame" params="camera_link_name camera_props">
+    <!-- need virtual joint due to axis misalignment -->
+    <link name="${camera_link_name}_virtual_link">
+      <visual>
+      </visual>
+    </link>
+    <joint type="fixed" name="${camera_link_name}_virtual_joint">
+      <origin rpy="${-pi/2} 0 ${-pi/2}" xyz="0 0 0"/>
+      <child link="${camera_link_name}_virtual_link"/>
+      <parent link="${camera_link_name}"/>
+    </joint>
     <gazebo reference="${camera_link_name}">
       <sensor name="${camera_link_name}_sensor" type="depth">
@@ -43,14 +53,8 @@
         <plugin name="depth_camera_controller" filename="libgazebo_ros_camera.so">
           <cameraName>${camera_link_name}</cameraName>
-          <imageTopicName>${camera_link_name}_ir/image_raw</imageTopicName>
-          <cameraInfoTopicName>${camera_link_name}_ir/camera_info</cameraInfoTopicName>
-          <depthImageTopicName>${camera_link_name}_depth/image_raw</depthImageTopicName>
-          <depthImageCameraInfoTopicName>${camera_link_name}_depth/camera_info</depthImageCameraInfoTopicName>
-          <pointCloudTopicName>${camera_link_name}_depth/points</pointCloudTopicName>
-          <frameName>${camera_link_name}_optical_frame</frameName>
+          <frame_name>${camera_link_name}_virtual_link</frame_name>
           <baseline>0.2</baseline>
           <alwaysOn>true</alwaysOn>
           <updateRate>0.0</updateRate>
-          <frame_name>camera_depth_frame</frame_name>
           <pointCloudCutoff>0.5</pointCloudCutoff>
           <pointCloudCutoffMax>3.0</pointCloudCutoffMax>

Commit message: Revert "costmap setup"

File: uwrt_mars_rover_drivetrain/uwrt_mars_rover_drivetrain_description/urdf/drivetrain.urdf.xacro (robot description, xacro)
@@ -48,7 +48,7 @@
   <xacro:generate_sensor_frame sensor_params="${sensors_parameters['depth_camera']['camera1']}" name="camera1"/>
   <xacro:default_depth_camera_frame camera_link_name="camera1" camera_props="${sensors_parameters['depth_camera']['camera1']['camera_properties']}"/>
-  <!-- <xacro:generate_sensor_frame sensor_params="${sensors_parameters['depth_camera']['camera2']}" name="camera2"/>
-  <xacro:default_depth_camera_frame camera_link_name="camera2" camera_props="${sensors_parameters['depth_camera']['camera2']['camera_properties']}"/> -->
-  <!-- <xacro:generate_sensor_frame sensor_params="${sensors_parameters['lidar']['lidar1']}"         name="lidar1"/>
-  <xacro:default_lidar_frame lidar_link_name="lidar1" lidar_props="${sensors_parameters['lidar']['lidar1']['lidar_properties']}"/> -->
+  <xacro:generate_sensor_frame sensor_params="${sensors_parameters['depth_camera']['camera2']}" name="camera2"/>
+  <xacro:default_depth_camera_frame camera_link_name="camera2" camera_props="${sensors_parameters['depth_camera']['camera2']['camera_properties']}"/>
+  <xacro:generate_sensor_frame sensor_params="${sensors_parameters['lidar']['lidar1']}"         name="lidar1"/>
+  <xacro:default_lidar_frame lidar_link_name="lidar1" lidar_props="${sensors_parameters['lidar']['lidar1']['lidar_properties']}"/>
 </robot>

File: uwrt_mars_rover_drivetrain/uwrt_mars_rover_drivetrain_description/urdf/sensors.macro.xacro (robot description, xacro)
@@ -25,14 +25,4 @@
   </xacro:macro>
   <xacro:macro name="default_depth_camera_frame" params="camera_link_name camera_props">
-    <!-- need virtual joint due to axis misalignment -->
-    <link name="${camera_link_name}_virtual_link">
-      <visual>
-      </visual>
-    </link>
-    <joint type="fixed" name="${camera_link_name}_virtual_joint">
-      <origin rpy="${-pi/2} 0 ${-pi/2}" xyz="0 0 0"/>
-      <child link="${camera_link_name}_virtual_link"/>
-      <parent link="${camera_link_name}"/>
-    </joint>
     <gazebo reference="${camera_link_name}">
       <sensor name="${camera_link_name}_sensor" type="depth">
@@ -53,8 +43,14 @@
         <plugin name="depth_camera_controller" filename="libgazebo_ros_camera.so">
           <cameraName>${camera_link_name}</cameraName>
-          <frame_name>${camera_link_name}_virtual_link</frame_name>
+          <imageTopicName>${camera_link_name}_ir/image_raw</imageTopicName>
+          <cameraInfoTopicName>${camera_link_name}_ir/camera_info</cameraInfoTopicName>
+          <depthImageTopicName>${camera_link_name}_depth/image_raw</depthImageTopicName>
+          <depthImageCameraInfoTopicName>${camera_link_name}_depth/camera_info</depthImageCameraInfoTopicName>
+          <pointCloudTopicName>${camera_link_name}_depth/points</pointCloudTopicName>
+          <frameName>${camera_link_name}_optical_frame</frameName>
           <baseline>0.2</baseline>
           <alwaysOn>true</alwaysOn>
           <updateRate>0.0</updateRate>
+          <frame_name>camera_depth_frame</frame_name>
           <pointCloudCutoff>0.5</pointCloudCutoff>
           <pointCloudCutoffMax>3.0</pointCloudCutoffMax>
