Commit message: xacro-ify ros2control urdf

File: uwrt_mars_rover_drivetrain/uwrt_mars_rover_drivetrain_description/urdf/drivetrain.macro.xacro (robot description, xacro)
@@ -2,15 +2,21 @@
 <robot xmlns:xacro="http://wiki.ros.org/xacro">
   <xacro:macro name="load_model_data" params="physical_parameters_file">
-    <!-- Read .yaml files and load contents into xacro properties -->
+    <!-- read .yaml files and load contents into xacro properties -->
     <xacro:property name="physical_parameters" value="${load_yaml(physical_parameters_file)}"/>
-    <!--  Extract data from yaml dictionaries  -->
+    <!--  extract data from yaml dictionaries  -->
     <xacro:property name="chassis_parameters" value="${physical_parameters['chassis']}"/>
     <xacro:property name="wheel_parameters" value="${physical_parameters['wheels']}"/>
+    <xacro:property name="control_parameters" value="${physical_parameters['control']}"/>
+    <!-- chassis parameters -->
     <xacro:property name="chassis_length" value="${chassis_parameters['length']}" scope="parent"/>
     <xacro:property name="chassis_width" value="${chassis_parameters['width']}" scope="parent"/>
     <xacro:property name="chassis_height" value="${chassis_parameters['height']}" scope="parent"/>
+    <!-- wheel parameters -->
     <xacro:property name="wheel_diameter" value="${wheel_parameters['diameter']}" scope="parent"/>
     <xacro:property name="wheel_width" value="${wheel_parameters['width']}" scope="parent"/>
     <xacro:property name="wheel_mass" value="${wheel_parameters['mass']}" scope="parent"/>
+    <!-- control parameters -->
+    <xacro:property name="mechanical_reduction" value="${control_parameters['mechanical_reduction']}" scope="parent"/>
+    <xacro:property name="max_speed" value="${control_parameters['max_speed']}" scope="parent"/>
   </xacro:macro>
   <xacro:macro name="default_inertial" params="mass:=5">
@@ -50,3 +56,25 @@
     </link>
   </xacro:macro>
+  <xacro:macro name="drivetrain_actuator" params="prefix suffix">
+    <ros2_control name="{prefix}_${suffix}_wheel_actuator" type="actuator">
+      <hardware>
+        <plugin>uwrt_mars_rover_drivetrain_hw/UWRTMarsRoverDrivetrainHardwareReal</plugin>
+        <!-- TODO: Can interface and Odrive id?-->
+      </hardware>
+      <joint name="${prefix}_${suffix}_wheel_joint">
+        <command_interface name="velocity">
+          <param name="min">"${-max_speed}"</param>
+          <param name="max">"${max_speed}"</param>
+        </command_interface>
+        <state_interface name="velocity"/>
+      </joint>
+      <transmission name="transmission1">
+        <!--  TODO: These are not actually parsed by ros2control yet: https://github.com/ros-controls/ros2_control/issues/32, https://github.com/ros-controls/ros2_control/issues/599 -->
+        <plugin>transmission_interface/SimpleTansmission</plugin>
+        <joint name="${prefix}_${suffix}_wheel_joint" role="joint1">
+          <mechanical_reduction>"${mechanical_reduction}"</mechanical_reduction>
+        </joint>
+      </transmission>
+    </ros2_control>
+  </xacro:macro>
 </robot>

File: uwrt_mars_rover_drivetrain/uwrt_mars_rover_drivetrain_description/urdf/drivetrain.urdf.xacro (robot description, xacro)
@@ -2,5 +2,5 @@
 <robot name="drivetrain" xmlns:xacro="http://www.ros.org/wiki/xacro">
   <!-- import macros file -->
-  <xacro:include filename="$(find uwrt_mars_rover_drivetrain_description)/urdf/common.xacro"/>
+  <xacro:include filename="$(find uwrt_mars_rover_drivetrain_description)/urdf/drivetrain.macro.xacro"/>
   <!-- load model data from yamls -->
   <xacro:load_model_data
@@ -8,4 +8,6 @@
   <!-- calculate parameters based on model data -->
   <xacro:property name="wheelbase_length" value="${chassis_width + wheel_width}"/>
+  <!-- include ros2control description -->
+  <xacro:include filename="$(find uwrt_mars_rover_drivetrain_description)/urdf/drivetrain.ros2control.xacro"/>
   <link name="base_link"/>
   <joint name="base_link_to_chassis" type="fixed">

Commit message: add gazebo launch

File: uwrt_mars_rover_drivetrain/uwrt_mars_rover_drivetrain_description/urdf/drivetrain.macro.xacro (robot description, xacro)
@@ -56,9 +56,14 @@
     </link>
   </xacro:macro>
-  <xacro:macro name="drivetrain_actuator" params="prefix suffix">
+  <xacro:macro name="drivetrain_actuator" params="prefix suffix sim_gazebo_classic:=^|false">
     <ros2_control name="${prefix}_${suffix}_wheel_actuator" type="actuator">
       <hardware>
+        <xacro:if value="${sim_gazebo_classic}">
+          <plugin>gazebo_ros2_control/GazeboSystem</plugin>
+        </xacro:if>
+        <xacro:unless value="${sim_gazebo_classic}">
         <plugin>uwrt_mars_rover_drivetrain_hw/UWRTMarsRoverDrivetrainHWActuatorInterface</plugin>
         <!-- TODO: CAN interface and Odrive id?-->
+        </xacro:unless>
       </hardware>
       <joint name="${prefix}_${suffix}_wheel_joint">

File: uwrt_mars_rover_drivetrain/uwrt_mars_rover_drivetrain_description/urdf/drivetrain.ros2control.xacro (robot description, xacro)
@@ -1,11 +1,25 @@
 <?xml version="1.0"?>
 <robot xmlns:xacro="http://www.ros.org/wiki/xacro">
+  <xacro:arg name="sim_gazebo_classic" default="true" />
   <!-- import macros file -->
   <xacro:include filename="$(find uwrt_mars_rover_drivetrain_description)/urdf/drivetrain.macro.xacro"/>
-  <xacro:drivetrain_actuator prefix="right" suffix="front"/>
-  <xacro:drivetrain_actuator prefix="right" suffix="middle"/>
-  <xacro:drivetrain_actuator prefix="right" suffix="back"/>
-  <xacro:drivetrain_actuator prefix="left" suffix="front"/>
-  <xacro:drivetrain_actuator prefix="left" suffix="middle"/>
-  <xacro:drivetrain_actuator prefix="left" suffix="back"/>
+  <xacro:drivetrain_actuator prefix="right" suffix="front" sim_gazebo_classic="$(arg sim_gazebo_classic)"/>
+  <xacro:drivetrain_actuator prefix="right" suffix="middle" sim_gazebo_classic="$(arg sim_gazebo_classic)"/>
+  <xacro:drivetrain_actuator prefix="right" suffix="back" sim_gazebo_classic="$(arg sim_gazebo_classic)"/>
+  <xacro:drivetrain_actuator prefix="left" suffix="front" sim_gazebo_classic="$(arg sim_gazebo_classic)"/>
+  <xacro:drivetrain_actuator prefix="left" suffix="middle" sim_gazebo_classic="$(arg sim_gazebo_classic)"/>
+  <xacro:drivetrain_actuator prefix="left" suffix="back" sim_gazebo_classic="$(arg sim_gazebo_classic)"/>
+  <xacro:if value="$(arg sim_gazebo_classic)">
+    <!-- Gazebo plugins -->
+    <gazebo reference="world">
+    </gazebo>
+    <gazebo>
+      <plugin filename="libgazebo_ros2_control.so" name="gazebo_ros2_control">
+      <robot_param>robot_description</robot_param>
+      <robot_param_node>robot_state_publisher</robot_param_node>
+      <robot_sim_type>gazebo_ros2_control/DefaultRobotHWSim</robot_sim_type>
+      <parameters>$(find uwrt_mars_rover_drivetrain_description)/config/drivetrain_controllers.yaml</parameters>
+      </plugin>
+    </gazebo>
+  </xacro:if>
 </robot>

Commit message: first time robot setup

File: uwrt_mars_rover_drivetrain/uwrt_mars_rover_drivetrain_description/urdf/drivetrain.macro.xacro (robot description, xacro)
@@ -36,4 +36,11 @@
       <xacro:insert_block name="identical_blocks"/>
     </collision>
+  </xacro:macro>
+  <xacro:macro name="box_inertia" params="m w h d">
+    <inertial>
+      <origin xyz="0 0 0" rpy="${pi/2} 0 ${pi/2}"/>
+      <mass value="${m}"/>
+      <inertia ixx="${(m/12) * (h*h + d*d)}" ixy="0.0" ixz="0.0" iyy="${(m/12) * (w*w + d*d)}" iyz="0.0" izz="${(m/12) * (w*w + h*h)}"/>
+    </inertial>
   </xacro:macro>
   <xacro:macro name="wheel" params="prefix suffix parent_link reflect wheel_diameter:=^ wheel_width:=^ wheel_mass:=^ wheelbase_length:=^ x_position" >

File: uwrt_mars_rover_drivetrain/uwrt_mars_rover_drivetrain_description/urdf/drivetrain.urdf.xacro (robot description, xacro)
@@ -26,4 +26,156 @@
     <xacro:default_inertial/>
   </link>
+  <link name="imu_link">
+    <visual>
+      <geometry>
+        <box size="0.1 0.1 0.1"/>
+      </geometry>
+    </visual>
+    <collision>
+      <geometry>
+        <box size="0.1 0.1 0.1"/>
+      </geometry>
+    </collision>
+    <xacro:box_inertia m="0.1" w="0.1" d="0.1" h="0.1"/>
+  </link>
+  <joint name="imu_joint" type="fixed">
+    <parent link="base_link"/>
+    <child link="imu_link"/>
+    <origin xyz="0 0 ${wheel_diameter/2}"/>
+  </joint>
+  <gazebo reference="imu_link">
+    <sensor name="imu_sensor" type="imu">
+      <plugin filename="libgazebo_ros_imu_sensor.so" name="imu_plugin">
+        <ros>
+          <namespace>/demo</namespace>
+          <remapping>~/out:=imu</remapping>
+        </ros>
+        <initial_orientation_as_reference>false</initial_orientation_as_reference>
+      </plugin>
+      <always_on>true</always_on>
+      <update_rate>100</update_rate>
+      <visualize>true</visualize>
+     <imu>
+     	<angular_velocity>
+     	  <x>
+     	    <noise type="gaussian">
+              <mean>0.0</mean>
+              <stddev>2e-4</stddev>
+              <bias_mean>0.0000075</bias_mean>
+              <bias_stddev>0.0000008</bias_stddev>
+            </noise>
+          </x>
+          <y>
+            <noise type="gaussian">
+              <mean>0.0</mean>
+              <stddev>2e-4</stddev>
+              <bias_mean>0.0000075</bias_mean>
+              <bias_stddev>0.0000008</bias_stddev>
+            </noise>
+          </y>
+          <z>
+            <noise type="gaussian">
+              <mean>0.0</mean>
+              <stddev>2e-4</stddev>
+              <bias_mean>0.0000075</bias_mean>
+              <bias_stddev>0.0000008</bias_stddev>
+            </noise>
+          </z>
+        </angular_velocity>
+        <linear_acceleration>
+          <x>
+            <noise type="gaussian">
+              <mean>0.0</mean>
+              <stddev>1.7e-2</stddev>
+              <bias_mean>0.1</bias_mean>
+              <bias_stddev>0.001</bias_stddev>
+            </noise>
+          </x>
+          <y>
+            <noise type="gaussian">
+              <mean>0.0</mean>
+              <stddev>1.7e-2</stddev>
+              <bias_mean>0.1</bias_mean>
+              <bias_stddev>0.001</bias_stddev>
+            </noise>
+          </y>
+          <z>
+            <noise type="gaussian">
+              <mean>0.0</mean>
+              <stddev>1.7e-2</stddev>
+              <bias_mean>0.1</bias_mean>
+              <bias_stddev>0.001</bias_stddev>
+            </noise>
+          </z>
+        </linear_acceleration>
+      </imu>
+    </sensor>
+  </gazebo>
+  <link name="camera_link">
+    <visual>
+      <origin xyz="0 0 0" rpy="0 0 0"/>
+      <geometry>
+        <box size="0.015 0.130 0.022"/>
+      </geometry>
+    </visual>
+    <collision>
+      <origin xyz="0 0 0" rpy="0 0 0"/>
+      <geometry>
+        <box size="0.015 0.130 0.022"/>
+      </geometry>
+    </collision>
+    <inertial>
+      <origin xyz="0 0 0" rpy="0 0 0"/>
+      <mass value="0.035"/>
+      <inertia ixx="0.001"  ixy="0"  ixz="0" iyy="0.001" iyz="0" izz="0.001" />
+    </inertial>
+  </link>
+  <joint name="camera_joint" type="fixed">
+    <parent link="base_link"/>
+    <child link="camera_link"/>
+    <origin xyz="0.215 0 0.05" rpy="0 0 0"/>
+  </joint>
+  <link name="camera_depth_frame"/>
+  <joint name="camera_depth_joint" type="fixed">
+    <origin xyz="0 0 0" rpy="${-pi/2} 0 ${-pi/2}"/>
+    <parent link="camera_link"/>
+    <child link="camera_depth_frame"/>
+  </joint>
+  <gazebo reference="camera_link">
+    <sensor name="depth_camera" type="depth">
+      <visualize>true</visualize>
+      <update_rate>30.0</update_rate>
+      <camera name="camera">
+        <horizontal_fov>1.047198</horizontal_fov>
+        <image>
+          <width>640</width>
+          <height>480</height>
+          <format>R8G8B8</format>
+        </image>
+        <clip>
+          <near>0.05</near>
+          <far>3</far>
+        </clip>
+      </camera>
+      <plugin name="depth_camera_controller" filename="libgazebo_ros_camera.so">
+        <baseline>0.2</baseline>
+        <alwaysOn>true</alwaysOn>
+        <updateRate>0.0</updateRate>
+        <frame_name>camera_depth_frame</frame_name>
+        <pointCloudCutoff>0.5</pointCloudCutoff>
+        <pointCloudCutoffMax>3.0</pointCloudCutoffMax>
+        <distortionK1>0</distortionK1>
+        <distortionK2>0</distortionK2>
+        <distortionK3>0</distortionK3>
+        <distortionT1>0</distortionT1>
+        <distortionT2>0</distortionT2>
+        <CxPrime>0</CxPrime>
+        <Cx>0</Cx>
+        <Cy>0</Cy>
+        <focalLength>0</focalLength>
+        <hackBaseline>0</hackBaseline>
+      </plugin>
+    </sensor>
+  </gazebo>
   <!-- wheels -->
   <xacro:wheel prefix="right" suffix="front" parent_link="chassis" reflect="-1" x_position="${chassis_length/2}"/>

Commit message: add can_ids to the hardware interface, commment out current stuff, clean up

File: uwrt_mars_rover_drivetrain/uwrt_mars_rover_drivetrain_description/urdf/drivetrain.macro.xacro (robot description, xacro)
@@ -56,9 +56,11 @@
     </link>
   </xacro:macro>
-  <xacro:macro name="drivetrain_actuator" params="prefix suffix">
+  <xacro:macro name="drivetrain_actuator" params="prefix suffix can_id">
+    <!-- convert the can_id argument to an xacro property -->
+    <xacro:property name="can_id_prop" value="${can_id}"/>
     <ros2_control name="${prefix}_${suffix}_wheel_actuator" type="actuator">
       <hardware>
         <plugin>uwrt_mars_rover_drivetrain_hw/UWRTMarsRoverDrivetrainHWActuatorInterface</plugin>
-        <!-- <param name="can_id" value="${can_id}"/> -->
+        <param name="can_id">${can_id_prop}</param>
         <!-- TODO: CAN interface?-->
       </hardware>
@@ -70,5 +72,5 @@
         <state_interface name="position"/>
         <state_interface name="velocity"/>
-        <state_interface name="iq_current"/>
+        <!-- <state_interface name="iq_current"/> -->
         <!-- TODO: acceleration, torque? -->
       </joint>

File: uwrt_mars_rover_drivetrain/uwrt_mars_rover_drivetrain_description/urdf/drivetrain.ros2control.xacro (robot description, xacro)
@@ -3,15 +3,9 @@
   <!-- import macros file -->
   <xacro:include filename="$(find uwrt_mars_rover_drivetrain_description)/urdf/drivetrain.macro.xacro"/>
-  <xacro:drivetrain_actuator prefix="right" suffix="front"/>
-  <xacro:drivetrain_actuator prefix="right" suffix="middle"/>
-  <xacro:drivetrain_actuator prefix="right" suffix="back"/>
-  <xacro:drivetrain_actuator prefix="left" suffix="front"/>
-  <xacro:drivetrain_actuator prefix="left" suffix="middle"/>
-  <xacro:drivetrain_actuator prefix="left" suffix="back"/>\
-  <!-- <xacro:drivetrain_actuator prefix="right" suffix="front" can_id="5"/>
+  <xacro:drivetrain_actuator prefix="right" suffix="front" can_id="5"/>
   <xacro:drivetrain_actuator prefix="right" suffix="middle" can_id="4"/>
   <xacro:drivetrain_actuator prefix="right" suffix="back" can_id="3"/>
   <xacro:drivetrain_actuator prefix="left" suffix="front" can_id="2"/>
   <xacro:drivetrain_actuator prefix="left" suffix="middle" can_id="1"/>
-  <xacro:drivetrain_actuator prefix="left" suffix="back" can_id="0"/> -->
+  <xacro:drivetrain_actuator prefix="left" suffix="back" can_id="0"/>
 </robot>

Commit message: loaded into gazebo

File: uwrt_mars_rover_drivetrain/uwrt_mars_rover_drivetrain_description/urdf/drivetrain.macro.xacro (robot description, xacro)
@@ -12,8 +12,10 @@
     <xacro:property name="chassis_width" value="${chassis_parameters['width']}" scope="parent"/>
     <xacro:property name="chassis_height" value="${chassis_parameters['height']}" scope="parent"/>
+    <xacro:property name="chassis_mass" value="${chassis_parameters['mass']}" scope="parent"/>
     <!-- wheel parameters -->
     <xacro:property name="wheel_diameter" value="${wheel_parameters['diameter']}" scope="parent"/>
     <xacro:property name="wheel_width" value="${wheel_parameters['width']}" scope="parent"/>
     <xacro:property name="wheel_mass" value="${wheel_parameters['mass']}" scope="parent"/>
+    <xacro:property name="wheel_radius" value="${(wheel_parameters['diameter'])/2}" scope="parent"/>
     <!-- control parameters -->
     <xacro:property name="mechanical_reduction" value="${control_parameters['mechanical_reduction']}" scope="parent"/>
@@ -27,4 +29,22 @@
           iyy="1e-3" iyz="0.0"
           izz="1e-3"/>
+    </inertial>
+  </xacro:macro>
+   <xacro:macro name="chassis_inertia" params="chassis_width:=^ chassis_height:=^ chassis_length:=^ chassis_mass:=^">
+    <inertial>
+      <mass value="${chassis_mass}" />
+      <inertia
+          ixx="${(1/12)*(((chassis_height)*(chassis_height))+((chassis_width)*(chassis_width)))}" ixy="0.0" ixz="0.0"
+          iyy="${(1/12)*(((chassis_height)*(chassis_height))+((chassis_length)*(chassis_length)))}" iyz="0.0"
+          izz="${(1/12)*(((chassis_width)*(chassis_width))+((chassis_length)*(chassis_length)))}"/>
+    </inertial>
+  </xacro:macro>
+  <xacro:macro name="wheel_intertia" params="wheel_radius:=^ wheel_width:=^ wheel_mass:=^">
+    <inertial>
+      <mass value="${wheel_mass}" />
+      <inertia
+          ixx="${(1/12)*(3*((wheel_radius)*(wheel_radius))+((wheel_width)*(wheel_width)))}" ixy="0.0" ixz="0.0"
+          iyy="${(1/12)*(3*((wheel_radius)*(wheel_radius))+((wheel_width)*(wheel_width)))}" iyz="0.0"
+          izz="${(1/2)*((wheel_radius)*(wheel_radius))}"/>
     </inertial>
   </xacro:macro>
@@ -53,5 +73,5 @@
         </idential_blocks>
       </xacro:identical_visual_collision>
-      <xacro:default_inertial mass="${wheel_mass}"/>
+      <xacro:wheel_intertia />
     </link>
   </xacro:macro>

File: uwrt_mars_rover_drivetrain/uwrt_mars_rover_drivetrain_description/urdf/drivetrain.urdf.xacro (robot description, xacro)
@@ -24,5 +24,5 @@
       </identical_blocks>
     </xacro:identical_visual_collision>
-    <xacro:default_inertial/>
+    <xacro:chassis_inertia/>
   </link>
   <!-- wheels -->

Commit message: User/nico-colin-keyon-andrew/can_drivetrain
Drivetrain ros2 control code for rover
---------

Co-authored-by: ColinToft <cwt1078@gmail.com>
Co-authored-by: Andrew Zhao <andrew2002zhao@gmail.com>
Co-authored-by: Keyon Jerome <keyonjerome@gmail.com>

File: uwrt_mars_rover_drivetrain/uwrt_mars_rover_drivetrain_description/urdf/drivetrain.macro.xacro (robot description, xacro)
@@ -56,9 +56,12 @@
     </link>
   </xacro:macro>
-  <xacro:macro name="drivetrain_actuator" params="prefix suffix">
+  <xacro:macro name="drivetrain_actuator" params="prefix suffix can_id">
+    <!-- convert the can_id argument to an xacro property -->
+    <xacro:property name="can_id_prop" value="${can_id}"/>
     <ros2_control name="${prefix}_${suffix}_wheel_actuator" type="actuator">
       <hardware>
         <plugin>uwrt_mars_rover_drivetrain_hw/UWRTMarsRoverDrivetrainHWActuatorInterface</plugin>
-        <!-- TODO: CAN interface and Odrive id?-->
+        <param name="can_id">${can_id_prop}</param>
+        <!-- TODO: CAN interface?-->
       </hardware>
       <joint name="${prefix}_${suffix}_wheel_joint">
@@ -69,5 +72,5 @@
         <state_interface name="position"/>
         <state_interface name="velocity"/>
-        <state_interface name="iq_current"/>
+        <!-- <state_interface name="iq_current"/> -->
         <!-- TODO: acceleration, torque? -->
       </joint>

File: uwrt_mars_rover_drivetrain/uwrt_mars_rover_drivetrain_description/urdf/drivetrain.ros2control.xacro (robot description, xacro)
@@ -3,9 +3,9 @@
   <!-- import macros file -->
   <xacro:include filename="$(find uwrt_mars_rover_drivetrain_description)/urdf/drivetrain.macro.xacro"/>
-  <xacro:drivetrain_actuator prefix="right" suffix="front"/>
-  <xacro:drivetrain_actuator prefix="right" suffix="middle"/>
-  <xacro:drivetrain_actuator prefix="right" suffix="back"/>
-  <xacro:drivetrain_actuator prefix="left" suffix="front"/>
-  <xacro:drivetrain_actuator prefix="left" suffix="middle"/>
-  <xacro:drivetrain_actuator prefix="left" suffix="back"/>
+  <xacro:drivetrain_actuator prefix="right" suffix="front" can_id="5"/>
+  <xacro:drivetrain_actuator prefix="right" suffix="middle" can_id="4"/>
+  <xacro:drivetrain_actuator prefix="right" suffix="back" can_id="3"/>
+  <xacro:drivetrain_actuator prefix="left" suffix="front" can_id="2"/>
+  <xacro:drivetrain_actuator prefix="left" suffix="middle" can_id="1"/>
+  <xacro:drivetrain_actuator prefix="left" suffix="back" can_id="0"/>
 </robot>
