Commit message: change macros and added params

File: uwrt_mars_rover_drivetrain/uwrt_mars_rover_drivetrain_description/urdf/drivetrain.macro.xacro (robot description, xacro)
@@ -57,4 +57,5 @@
     </collision>
   </xacro:macro>
+  <!-- macro for the wheel -->
   <xacro:macro name="wheel" params="prefix suffix parent_link reflect wheel_diameter:=^ wheel_width:=^ wheel_mass:=^ wheelbase_length:=^ x_position" >
     <joint name="${prefix}_${suffix}_wheel_joint" type="continuous">
@@ -76,4 +77,16 @@
     </link>
   </xacro:macro>
+  <!-- drivetrain macro only for the simulation stuff -->
+  <xacro:macro name="drivetrain_actuator_gazebo" params="prefix suffix">
+      <joint name="${prefix}_${suffix}_wheel_joint">
+        <command_interface name="velocity">
+          <param name="min">${-max_speed}</param>
+          <param name="max">${max_speed}</param>
+        </command_interface>
+        <state_interface name="position"/>
+        <state_interface name="velocity"/>
+      </joint>
+  </xacro:macro>
+  <!-- actual hardware -->
   <xacro:macro name="drivetrain_actuator" params="prefix suffix can_id">
     <!-- convert the can_id argument to an xacro property -->
@@ -103,9 +116,4 @@
       </transmission> -->
     </ros2_control>
-      <gazebo>
-        <plugin filename="libgazebo_ros2_control.so" name="gazebo_ros2_control">
-          <parameters>$(find uwrt_mars_rover_drivetrain_hw)/config/drivetrain_controllers.yaml</parameters>
-        </plugin>
-      </gazebo>
   </xacro:macro>
 </robot>

File: uwrt_mars_rover_drivetrain/uwrt_mars_rover_drivetrain_description/urdf/drivetrain.urdf.xacro (robot description, xacro)
@@ -3,4 +3,5 @@
   <!-- import macros file -->
   <xacro:include filename="$(find uwrt_mars_rover_drivetrain_description)/urdf/drivetrain.macro.xacro"/>
+  <xacro:arg name="sim" default="false"/>
   <!-- load model data from yamls -->
   <xacro:load_model_data
@@ -8,6 +9,12 @@
   <!-- calculate parameters based on model data -->
   <xacro:property name="wheelbase_length" value="${chassis_width + wheel_width}"/>
-  <!-- include ros2control description -->
-  <xacro:include filename="$(find uwrt_mars_rover_drivetrain_description)/urdf/drivetrain.ros2control.xacro"/>
+  <!-- include ros2control description for regular -->
+  <xacro:unless value="$(arg sim)">
+      <xacro:include filename="$(find uwrt_mars_rover_drivetrain_description)/urdf/drivetrain.ros2control.xacro"/>
+  </xacro:unless>
+  <!-- include ros2 control for sim -->
+  <xacro:if value="$(arg sim)">
+      <xacro:include filename="$(find uwrt_mars_rover_drivetrain_description)/urdf/drivetrain.ros2controlgazebo.xacro"/>
+  </xacro:if>
   <link name="base_link"/>
   <joint name="base_link_to_chassis" type="fixed">
@@ -26,10 +33,10 @@
     <xacro:chassis_inertia/>
   </link>
-  <!-- wheels -->
-  <xacro:wheel prefix="right" suffix="front" parent_link="chassis" reflect="-1" x_position="${chassis_length/2}"/>
-  <xacro:wheel prefix="right" suffix="middle" parent_link="chassis" reflect="-1" x_position="0"/>
-  <xacro:wheel prefix="right" suffix="back" parent_link="chassis" reflect="-1" x_position="${-chassis_length/2}"/>
-  <xacro:wheel prefix="left" suffix="front" parent_link="chassis" reflect="1" x_position="${chassis_length/2}"/>
-  <xacro:wheel prefix="left" suffix="middle" parent_link="chassis" reflect="1" x_position="0"/>
-  <xacro:wheel prefix="left" suffix="back" parent_link="chassis" reflect="1" x_position="${-chassis_length/2}"/>
+    <!-- wheels -->
+    <xacro:wheel prefix="right" suffix="front" parent_link="chassis" reflect="-1" x_position="${chassis_length/2}"/>
+    <xacro:wheel prefix="right" suffix="middle" parent_link="chassis" reflect="-1" x_position="0"/>
+    <xacro:wheel prefix="right" suffix="back" parent_link="chassis" reflect="-1" x_position="${-chassis_length/2}"/>
+    <xacro:wheel prefix="left" suffix="front" parent_link="chassis" reflect="1" x_position="${chassis_length/2}"/>
+    <xacro:wheel prefix="left" suffix="middle" parent_link="chassis" reflect="1" x_position="0"/>
+    <xacro:wheel prefix="left" suffix="back" parent_link="chassis" reflect="1" x_position="${-chassis_length/2}"/>
 </robot>

Commit message: basic imu urdf setup

File: uwrt_mars_rover_drivetrain/uwrt_mars_rover_drivetrain_description/urdf/drivetrain.macro.xacro (robot description, xacro)
@@ -104,3 +104,91 @@
     </ros2_control>
   </xacro:macro>
+  <xacro:macro name="nav_imu">
+    <link name="nav_imu_link">
+      <visual>
+        <geometry>
+          <box size="0.1 0.1 0.1"/>
+        </geometry>
+      </visual>
+      <collision>
+        <geometry>
+          <box size="0.1 0.1 0.1"/>
+        </geometry>
+      </collision>
+      <!-- <xacro:box_inertia m="0.1" w="0.1" d="0.1" h="0.1"/> -->
+    </link>
+    <joint name="nav_imu_joint" type="fixed">
+      <parent link="base_link"/>
+      <child link="nav_imu_link"/>
+      <origin xyz="0 0 0.01"/>
+    </joint>
+    <gazebo reference="nav_imu_link">
+      <sensor name="nav_imu_sensor" type="imu">
+       <plugin filename="libgazebo_ros_imu_sensor.so" name="imu_plugin">
+          <ros>
+            <namespace>/demo</namespace>
+            <remapping>~/out:=imu</remapping>
+          </ros>
+          <initial_orientation_as_reference>false</initial_orientation_as_reference>
+        </plugin>
+        <always_on>true</always_on>
+        <update_rate>100</update_rate>
+        <visualize>true</visualize>
+        <imu>
+          <angular_velocity>
+            <x>
+              <noise type="gaussian">
+                <mean>0.0</mean>
+                <stddev>2e-4</stddev>
+                <bias_mean>0.0000075</bias_mean>
+                <bias_stddev>0.0000008</bias_stddev>
+              </noise>
+            </x>
+            <y>
+              <noise type="gaussian">
+                <mean>0.0</mean>
+                <stddev>2e-4</stddev>
+                <bias_mean>0.0000075</bias_mean>
+                <bias_stddev>0.0000008</bias_stddev>
+              </noise>
+            </y>
+            <z>
+              <noise type="gaussian">
+                <mean>0.0</mean>
+                <stddev>2e-4</stddev>
+                <bias_mean>0.0000075</bias_mean>
+                <bias_stddev>0.0000008</bias_stddev>
+              </noise>
+            </z>
+          </angular_velocity>
+          <linear_acceleration>
+            <x>
+              <noise type="gaussian">
+                <mean>0.0</mean>
+                <stddev>1.7e-2</stddev>
+                <bias_mean>0.1</bias_mean>
+                <bias_stddev>0.001</bias_stddev>
+              </noise>
+            </x>
+            <y>
+              <noise type="gaussian">
+                <mean>0.0</mean>
+                <stddev>1.7e-2</stddev>
+                <bias_mean>0.1</bias_mean>
+                <bias_stddev>0.001</bias_stddev>
+              </noise>
+            </y>
+            <z>
+              <noise type="gaussian">
+                <mean>0.0</mean>
+                <stddev>1.7e-2</stddev>
+                <bias_mean>0.1</bias_mean>
+                <bias_stddev>0.001</bias_stddev>
+              </noise>
+            </z>
+          </linear_acceleration>
+        </imu>
+      </sensor>
+    </gazebo>
+  </xacro:macro>
 </robot>

File: uwrt_mars_rover_drivetrain/uwrt_mars_rover_drivetrain_description/urdf/drivetrain.urdf.xacro (robot description, xacro)
@@ -33,3 +33,4 @@
   <xacro:wheel prefix="left" suffix="middle" parent_link="chassis" reflect="1" x_position="0"/>
   <xacro:wheel prefix="left" suffix="back" parent_link="chassis" reflect="1" x_position="${-chassis_length/2}"/>
+  <xacro:nav_imu/>
 </robot>

Commit message: add gps setup (untested)

File: uwrt_mars_rover_drivetrain/uwrt_mars_rover_drivetrain_description/urdf/drivetrain.macro.xacro (robot description, xacro)
@@ -110,4 +110,7 @@
           <box size="0.1 0.1 0.1"/>
         </geometry>
+        <!-- <material name="cyan"> -->
+        <!--   <color rgba"0 1.0 1.0 1.0"/> -->
+        <!-- </material> -->
       </visual>
       <collision>
@@ -125,5 +128,5 @@
     <gazebo reference="nav_imu_link">
       <sensor name="nav_imu_sensor" type="imu">
-       <plugin filename="libgazebo_ros_imu_sensor.so" name="imu_plugin">
+       <plugin filename="libgazebo_ros_imu_sensor.so" name="nav_imu_plugin">
           <ros>
             <namespace>/demo</namespace>
@@ -192,3 +195,40 @@
     </gazebo>
   </xacro:macro>
+  <xacro:macro name="nav_gps">
+    <link name="nav_gps_link">
+      <visual>
+        <geometry>
+          <box size="0.1 0.1 0.1"/>
+        </geometry>
+        <!-- <material name="cyan"> -->
+        <!--   <color rgba"0 1.0 1.0 1.0"/> -->
+        <!-- </material> -->
+      </visual>
+      <collision>
+        <geometry>
+          <box size="0.1 0.1 0.1"/>
+        </geometry>
+      </collision>
+      <!-- <xacro:box_inertia m="0.1" w="0.1" d="0.1" h="0.1"/> -->
+    </link>
+    <joint name="nav_gps_joint" type="fixed">
+      <parent link="base_link"/>
+      <child link="nav_gps_link"/>
+      <origin xyz="0 0 0.01"/>
+    </joint>
+    <gazebo reference="nav_gps_link">
+        <sensor name="nav_gps_sensor" type="gps">
+            <always_on>true</always_on>
+            <update_rate>1.0</update_rate>
+            <plugin name="nav_gps_plugin" filename="libgazebo_ros_gps_sensor.so">
+                <ros>
+                    <!-- <namespace>/br</namespace> -->
+                    <remapping>nav_gps_plugin/out:=gps</remapping>
+                </ros>
+                <frame_name>gps_link</frame_name>
+            </plugin>
+        </sensor>
+        <material>Gazebo/Grey</material> <!-- TODO: fix? --!>
+    </gazebo>
+  </xacro:macro>
 </robot>

Commit message: added gps setup (publishes)

File: uwrt_mars_rover_drivetrain/uwrt_mars_rover_drivetrain_description/urdf/drivetrain.macro.xacro (robot description, xacro)
@@ -128,5 +128,5 @@
     <gazebo reference="nav_imu_link">
       <sensor name="nav_imu_sensor" type="imu">
-       <plugin filename="libgazebo_ros_imu_sensor.so" name="nav_imu_plugin">
+       <plugin filename="libgazebo_ros_imu_sensor.so" name="imu_plugin">
           <ros>
             <namespace>/demo</namespace>
@@ -219,15 +219,30 @@
     <gazebo reference="nav_gps_link">
         <sensor name="nav_gps_sensor" type="gps">
-            <always_on>true</always_on>
-            <update_rate>1.0</update_rate>
             <plugin name="nav_gps_plugin" filename="libgazebo_ros_gps_sensor.so">
                 <ros>
-                    <!-- <namespace>/br</namespace> -->
-                    <remapping>nav_gps_plugin/out:=gps</remapping>
+                  <namespace>/demo</namespace>
+                    <remapping>~/out:=gps</remapping>
                 </ros>
                 <frame_name>gps_link</frame_name>
             </plugin>
+            <always_on>true</always_on>
+            <update_rate>100</update_rate>
+            <visualize>true</visualize>
+            <gps>
+              <longitude>
+                  <mean>0.0</mean>
+                  <stddev>2e-4</stddev>
+                  <bias_mean>0.0000075</bias_mean>
+                  <bias_stddev>0.0000008</bias_stddev>
+              </longitude>
+              <latitude>
+                  <mean>0.0</mean>
+                  <stddev>2e-4</stddev>
+                  <bias_mean>0.0000075</bias_mean>
+                  <bias_stddev>0.0000008</bias_stddev>
+              </latitude>
+            </gps>
         </sensor>
-        <material>Gazebo/Grey</material> <!-- TODO: fix? --!>
+        <material>Gazebo/Grey</material> <!-- TODO: fix? -->
     </gazebo>
   </xacro:macro>

File: uwrt_mars_rover_drivetrain/uwrt_mars_rover_drivetrain_description/urdf/drivetrain.urdf.xacro (robot description, xacro)
@@ -34,3 +34,4 @@
   <xacro:wheel prefix="left" suffix="back" parent_link="chassis" reflect="1" x_position="${-chassis_length/2}"/>
   <xacro:nav_imu/>
+  <xacro:nav_gps/>
 </robot>

Commit message: physical and sim works

File: uwrt_mars_rover_drivetrain/uwrt_mars_rover_drivetrain_description/urdf/drivetrain.macro.xacro (robot description, xacro)
@@ -94,5 +94,5 @@
     <ros2_control name="${prefix}_${suffix}_wheel_actuator" type="actuator">
       <hardware>
-        <plugin>gazebo_ros2_control/GazeboSystem</plugin>
+        <plugin>uwrt_mars_rover_drivetrain_hw/UWRTMarsRoverDrivetrainHWActuatorInterface</plugin>
         <param name="can_id">${can_id_prop}</param>
         <!-- TODO: CAN interface?-->
@@ -109,10 +109,10 @@
       </joint>
       <!-- <transmission name="transmission1"> -->
-        <!--  TODO: These are not actually parsed by ros2control yet: https://github.com/ros-controls/ros2_control/issues/32, https://github.com/ros-controls/ros2_control/issues/599 -->
-        <!-- <plugin>transmission_interface/SimpleTransmission</plugin>
-        <joint name="${prefix}_${suffix}_wheel_joint" role="joint1">
-          <mechanical_reduction>${mechanical_reduction}</mechanical_reduction>
-        </joint>
-      </transmission> -->
+         <!-- TODO: These are not actually parsed by ros2control yet: https://github.com/ros-controls/ros2_control/issues/32, https://github.com/ros-controls/ros2_control/issues/599 -->
+        <!-- <plugin>transmission_interface/SimpleTransmission</plugin> -->
+        <!-- <joint name="${prefix}_${suffix}_wheel_joint" role="joint1"> -->
+          <!-- <mechanical_reduction>${mechanical_reduction}</mechanical_reduction> -->
+        <!-- </joint> -->
+      <!-- </transmission> -->
     </ros2_control>
   </xacro:macro>

File: uwrt_mars_rover_drivetrain/uwrt_mars_rover_drivetrain_description/urdf/drivetrain.ros2controlgazebo.xacro (robot description, xacro)
@@ -3,5 +3,5 @@
   <!-- import macros file -->
   <xacro:include filename="$(find uwrt_mars_rover_drivetrain_description)/urdf/drivetrain.macro.xacro"/>
-  <xacro:macro name="uwrt_drivetrain_ros2_controls">
+  <xacro:macro name="uwrt_drivetrain_ros2_controls_gazebo">
     <ros2_control name="gazebo_wheel_actuator" type="system">
       <hardware>

File: uwrt_mars_rover_drivetrain/uwrt_mars_rover_drivetrain_description/urdf/drivetrain.urdf.xacro (robot description, xacro)
@@ -12,8 +12,10 @@
   <xacro:if value="$(arg sim)">
       <xacro:include filename="$(find uwrt_mars_rover_drivetrain_description)/urdf/drivetrain.ros2controlgazebo.xacro"/>
+      <xacro:uwrt_drivetrain_ros2_controls_gazebo/>
   </xacro:if>
   <!-- include ros2control description for regular -->
   <xacro:unless value="$(arg sim)">
       <xacro:include filename="$(find uwrt_mars_rover_drivetrain_description)/urdf/drivetrain.ros2control.xacro"/>
+      <xacro:uwrt_drivetrain_ros2_controls/>
   </xacro:unless>
   <link name="base_link"/>
@@ -40,4 +42,3 @@
   <xacro:wheel prefix="left" suffix="middle" parent_link="chassis" reflect="1" x_position="0"/>
   <xacro:wheel prefix="left" suffix="back" parent_link="chassis" reflect="1" x_position="${-chassis_length/2}"/>
-  <xacro:uwrt_drivetrain_ros2_controls/>
 </robot>

Commit message: cherry picked commit into sim 2024

File: uwrt_mars_rover_drivetrain/uwrt_mars_rover_drivetrain_description/urdf/drivetrain.macro.xacro (robot description, xacro)
@@ -57,4 +57,5 @@
     </collision>
   </xacro:macro>
+  <!-- macro for the wheel -->
   <xacro:macro name="wheel" params="prefix suffix parent_link reflect wheel_diameter:=^ wheel_width:=^ wheel_mass:=^ wheelbase_length:=^ x_position" >
     <joint name="${prefix}_${suffix}_wheel_joint" type="continuous">
@@ -76,4 +77,16 @@
     </link>
   </xacro:macro>
+  <!-- drivetrain macro only for the simulation stuff -->
+  <xacro:macro name="drivetrain_actuator_gazebo" params="prefix suffix">
+      <joint name="${prefix}_${suffix}_wheel_joint">
+        <command_interface name="velocity">
+          <param name="min">${-max_speed}</param>
+          <param name="max">${max_speed}</param>
+        </command_interface>
+        <state_interface name="position"/>
+        <state_interface name="velocity"/>
+      </joint>
+  </xacro:macro>
+  <!-- actual hardware -->
   <xacro:macro name="drivetrain_actuator" params="prefix suffix can_id">
     <!-- convert the can_id argument to an xacro property -->
@@ -95,11 +108,11 @@
         <!-- TODO: acceleration, torque? -->
       </joint>
-      <transmission name="transmission1">
-        <!--  TODO: These are not actually parsed by ros2control yet: https://github.com/ros-controls/ros2_control/issues/32, https://github.com/ros-controls/ros2_control/issues/599 -->
-        <plugin>transmission_interface/SimpleTransmission</plugin>
-        <joint name="${prefix}_${suffix}_wheel_joint" role="joint1">
-          <mechanical_reduction>${mechanical_reduction}</mechanical_reduction>
-        </joint>
-      </transmission>
+      <!-- <transmission name="transmission1"> -->
+         <!-- TODO: These are not actually parsed by ros2control yet: https://github.com/ros-controls/ros2_control/issues/32, https://github.com/ros-controls/ros2_control/issues/599 -->
+        <!-- <plugin>transmission_interface/SimpleTransmission</plugin> -->
+        <!-- <joint name="${prefix}_${suffix}_wheel_joint" role="joint1"> -->
+          <!-- <mechanical_reduction>${mechanical_reduction}</mechanical_reduction> -->
+        <!-- </joint> -->
+      <!-- </transmission> -->
     </ros2_control>
   </xacro:macro>

File: uwrt_mars_rover_drivetrain/uwrt_mars_rover_drivetrain_description/urdf/drivetrain.urdf.xacro (robot description, xacro)
@@ -4,4 +4,5 @@
   <xacro:include filename="$(find uwrt_mars_rover_drivetrain_description)/urdf/drivetrain.macro.xacro"/>
   <xacro:include filename="$(find uwrt_mars_rover_drivetrain_description)/urdf/sensors.macro.xacro"/>
+  <xacro:arg name="sim" default="true"/>
   <!-- load model data from yamls -->
   <xacro:load_model_data
@@ -10,12 +11,15 @@
   <!-- calculate parameters based on model data -->
   <xacro:property name="wheelbase_length" value="${chassis_width + wheel_width}"/>
-  <!-- include ros2control description -->
-  <xacro:include filename="$(find uwrt_mars_rover_drivetrain_description)/urdf/drivetrain.ros2control.xacro"/>
+    <!-- include ros2 control for sim -->
+  <xacro:if value="$(arg sim)">
+      <xacro:include filename="$(find uwrt_mars_rover_drivetrain_description)/urdf/drivetrain.ros2controlgazebo.xacro"/>
+      <xacro:uwrt_drivetrain_ros2_controls_gazebo/>
+  </xacro:if>
+  <!-- include ros2control description for regular -->
+  <xacro:unless value="$(arg sim)">
+      <xacro:include filename="$(find uwrt_mars_rover_drivetrain_description)/urdf/drivetrain.ros2control.xacro"/>
+      <xacro:uwrt_drivetrain_ros2_controls/>
+  </xacro:unless>
   <link name="base_link"/>
-  <joint name="base_link_to_chassis" type="fixed">
-    <parent link="base_link"/>
-    <child link="chassis"/>
-    <origin xyz="0 0 ${wheel_diameter/2}" rpy="0 0 0"/>
-  </joint>
   <link name="chassis">
     <xacro:identical_visual_collision>
@@ -28,4 +32,9 @@
     <xacro:chassis_inertia/>
   </link>
+  <joint name="base_link_to_chassis" type="fixed">
+    <parent link="base_link"/>
+    <child link="chassis"/>
+    <origin xyz="0 0 ${wheel_diameter/2}" rpy="0 0 0"/>
+  </joint>
   <!-- wheels -->
   <xacro:wheel prefix="right" suffix="front" parent_link="chassis" reflect="-1" x_position="${chassis_length/2}"/>
