Commit message: squashed commits

File: uwrt_mars_rover_drivetrain/uwrt_mars_rover_drivetrain_description/urdf/drivetrain.macro.xacro (robot description, xacro)
@@ -12,8 +12,10 @@
     <xacro:property name="chassis_width" value="${chassis_parameters['width']}" scope="parent"/>
     <xacro:property name="chassis_height" value="${chassis_parameters['height']}" scope="parent"/>
+    <xacro:property name="chassis_mass" value="${chassis_parameters['mass']}" scope="parent"/>
     <!-- wheel parameters -->
     <xacro:property name="wheel_diameter" value="${wheel_parameters['diameter']}" scope="parent"/>
     <xacro:property name="wheel_width" value="${wheel_parameters['width']}" scope="parent"/>
     <xacro:property name="wheel_mass" value="${wheel_parameters['mass']}" scope="parent"/>
+    <xacro:property name="wheel_radius" value="${(wheel_parameters['diameter'])/2}" scope="parent"/>
     <!-- control parameters -->
     <xacro:property name="mechanical_reduction" value="${control_parameters['mechanical_reduction']}" scope="parent"/>
@@ -29,4 +31,22 @@
     </inertial>
   </xacro:macro>
+   <xacro:macro name="chassis_inertia" params="chassis_width:=^ chassis_height:=^ chassis_length:=^ chassis_mass:=^">
+    <inertial>
+      <mass value="${chassis_mass}" />
+      <inertia
+          ixx="${(1/12)*(((chassis_height)*(chassis_height))+((chassis_width)*(chassis_width)))}" ixy="0.0" ixz="0.0"
+          iyy="${(1/12)*(((chassis_height)*(chassis_height))+((chassis_length)*(chassis_length)))}" iyz="0.0"
+          izz="${(1/12)*(((chassis_width)*(chassis_width))+((chassis_length)*(chassis_length)))}"/>
+    </inertial>
+  </xacro:macro>
+  <xacro:macro name="wheel_intertia" params="wheel_radius:=^ wheel_width:=^ wheel_mass:=^">
+    <inertial>
+      <mass value="${wheel_mass}" />
+      <inertia
+          ixx="${(1/12)*(3*((wheel_radius)*(wheel_radius))+((wheel_width)*(wheel_width)))}" ixy="0.0" ixz="0.0"
+          iyy="${(1/12)*(3*((wheel_radius)*(wheel_radius))+((wheel_width)*(wheel_width)))}" iyz="0.0"
+          izz="${(1/2)*((wheel_radius)*(wheel_radius))}"/>
+    </inertial>
+  </xacro:macro>
   <xacro:macro name="identical_visual_collision" params="**identical_blocks">
     <visual>
@@ -37,4 +57,5 @@
     </collision>
   </xacro:macro>
+  <!-- macro for the wheel -->
   <xacro:macro name="wheel" params="prefix suffix parent_link reflect wheel_diameter:=^ wheel_width:=^ wheel_mass:=^ wheelbase_length:=^ x_position" >
     <joint name="${prefix}_${suffix}_wheel_joint" type="continuous">
@@ -53,7 +74,19 @@
         </idential_blocks>
       </xacro:identical_visual_collision>
-      <xacro:default_inertial mass="${wheel_mass}"/>
+      <xacro:wheel_intertia />
     </link>
   </xacro:macro>
+  <!-- drivetrain macro only for the simulation stuff -->
+  <xacro:macro name="drivetrain_actuator_gazebo" params="prefix suffix">
+      <joint name="${prefix}_${suffix}_wheel_joint">
+        <command_interface name="velocity">
+          <param name="min">${-max_speed}</param>
+          <param name="max">${max_speed}</param>
+        </command_interface>
+        <state_interface name="position"/>
+        <state_interface name="velocity"/>
+      </joint>
+  </xacro:macro>
+  <!-- actual hardware -->
   <xacro:macro name="drivetrain_actuator" params="prefix suffix can_id">
     <!-- convert the can_id argument to an xacro property -->
@@ -75,11 +108,11 @@
         <!-- TODO: acceleration, torque? -->
       </joint>
-      <transmission name="transmission1">
-        <!--  TODO: These are not actually parsed by ros2control yet: https://github.com/ros-controls/ros2_control/issues/32, https://github.com/ros-controls/ros2_control/issues/599 -->
-        <plugin>transmission_interface/SimpleTransmission</plugin>
-        <joint name="${prefix}_${suffix}_wheel_joint" role="joint1">
-          <mechanical_reduction>${mechanical_reduction}</mechanical_reduction>
-        </joint>
-      </transmission>
+      <!-- <transmission name="transmission1"> -->
+         <!-- TODO: These are not actually parsed by ros2control yet: https://github.com/ros-controls/ros2_control/issues/32, https://github.com/ros-controls/ros2_control/issues/599 -->
+        <!-- <plugin>transmission_interface/SimpleTransmission</plugin> -->
+        <!-- <joint name="${prefix}_${suffix}_wheel_joint" role="joint1"> -->
+          <!-- <mechanical_reduction>${mechanical_reduction}</mechanical_reduction> -->
+        <!-- </joint> -->
+      <!-- </transmission> -->
     </ros2_control>
   </xacro:macro>

File: uwrt_mars_rover_drivetrain/uwrt_mars_rover_drivetrain_description/urdf/drivetrain.ros2control.xacro (robot description, xacro)
@@ -3,9 +3,11 @@
   <!-- import macros file -->
   <xacro:include filename="$(find uwrt_mars_rover_drivetrain_description)/urdf/drivetrain.macro.xacro"/>
-  <xacro:drivetrain_actuator prefix="right" suffix="front" can_id="5"/>
-  <xacro:drivetrain_actuator prefix="right" suffix="middle" can_id="4"/>
-  <xacro:drivetrain_actuator prefix="right" suffix="back" can_id="3"/>
-  <xacro:drivetrain_actuator prefix="left" suffix="front" can_id="2"/>
-  <xacro:drivetrain_actuator prefix="left" suffix="middle" can_id="1"/>
-  <xacro:drivetrain_actuator prefix="left" suffix="back" can_id="0"/>
+  <xacro:macro name="uwrt_drivetrain_ros2_controls">
+    <xacro:drivetrain_actuator prefix="right" suffix="front" can_id="5"/>
+    <xacro:drivetrain_actuator prefix="right" suffix="middle" can_id="4"/>
+    <xacro:drivetrain_actuator prefix="right" suffix="back" can_id="3"/>
+    <xacro:drivetrain_actuator prefix="left" suffix="front" can_id="2"/>
+    <xacro:drivetrain_actuator prefix="left" suffix="middle" can_id="1"/>
+    <xacro:drivetrain_actuator prefix="left" suffix="back" can_id="0"/>
+ </xacro:macro>
 </robot>

Commit message: localization changes with gps and imu

File: uwrt_mars_rover_drivetrain/uwrt_mars_rover_drivetrain_description/urdf/drivetrain.macro.xacro (robot description, xacro)
@@ -29,5 +29,5 @@
           iyy="1e-3" iyz="0.0"
           izz="1e-3"/>
-    </inertial>
+      </inertial>
   </xacro:macro>
    <xacro:macro name="chassis_inertia" params="chassis_width:=^ chassis_height:=^ chassis_length:=^ chassis_mass:=^">
@@ -132,17 +132,13 @@
         </geometry>
       </collision>
+      <xacro:default_inertial mass="0.001"/>
       <!-- <xacro:box_inertia m="0.1" w="0.1" d="0.1" h="0.1"/> -->
     </link>
-    <joint name="nav_imu_joint" type="fixed">
-      <parent link="base_link"/>
-      <child link="nav_imu_link"/>
-      <origin xyz="0 0 0.01"/>
-    </joint>
     <gazebo reference="nav_imu_link">
       <sensor name="nav_imu_sensor" type="imu">
        <plugin filename="libgazebo_ros_imu_sensor.so" name="imu_plugin">
           <ros>
-            <namespace>/demo</namespace>
-            <remapping>~/out:=imu</remapping>
+            <!-- <namespace>/demo</namespace> -->
+            <remapping>~/out:=imu/data</remapping>
           </ros>
           <initial_orientation_as_reference>false</initial_orientation_as_reference>
@@ -157,6 +153,6 @@
                 <mean>0.0</mean>
                 <stddev>2e-4</stddev>
-                <bias_mean>0.0000075</bias_mean>
-                <bias_stddev>0.0000008</bias_stddev>
+                <!-- <bias_mean>0.0000075</bias_mean>
+                <bias_stddev>0.0000008</bias_stddev> -->
               </noise>
             </x>
@@ -165,6 +161,6 @@
                 <mean>0.0</mean>
                 <stddev>2e-4</stddev>
-                <bias_mean>0.0000075</bias_mean>
-                <bias_stddev>0.0000008</bias_stddev>
+                <!-- <bias_mean>0.0000075</bias_mean>
+                <bias_stddev>0.0000008</bias_stddev> -->
               </noise>
             </y>
@@ -173,6 +169,6 @@
                 <mean>0.0</mean>
                 <stddev>2e-4</stddev>
-                <bias_mean>0.0000075</bias_mean>
-                <bias_stddev>0.0000008</bias_stddev>
+                <!-- <bias_mean>0.0000075</bias_mean>
+                <bias_stddev>0.0000008</bias_stddev> -->
               </noise>
             </z>
@@ -183,6 +179,6 @@
                 <mean>0.0</mean>
                 <stddev>1.7e-2</stddev>
-                <bias_mean>0.1</bias_mean>
-                <bias_stddev>0.001</bias_stddev>
+                <!-- <bias_mean>0.1</bias_mean>
+                <bias_stddev>0.001</bias_stddev> -->
               </noise>
             </x>
@@ -191,6 +187,6 @@
                 <mean>0.0</mean>
                 <stddev>1.7e-2</stddev>
-                <bias_mean>0.1</bias_mean>
-                <bias_stddev>0.001</bias_stddev>
+                <!-- <bias_mean>0.1</bias_mean>
+                <bias_stddev>0.001</bias_stddev> -->
               </noise>
             </y>
@@ -199,6 +195,6 @@
                 <mean>0.0</mean>
                 <stddev>1.7e-2</stddev>
-                <bias_mean>0.1</bias_mean>
-                <bias_stddev>0.001</bias_stddev>
+                <!-- <bias_mean>0.1</bias_mean>
+                <bias_stddev>0.001</bias_stddev> -->
               </noise>
             </z>
@@ -207,7 +203,15 @@
       </sensor>
     </gazebo>
+    <joint name="nav_imu_joint" type="fixed">
+      <parent link="base_link"/>
+      <child link="nav_imu_link"/>
+      <origin xyz ="0 0 0.01"/>
+      <axis>
+          <xyz>0 0 1</xyz>
+      </axis>
+    </joint>
   </xacro:macro>
   <xacro:macro name="nav_gps">
-    <link name="nav_gps_link">
+    <link name="gps_link">
       <visual>
         <geometry>
@@ -223,17 +227,13 @@
         </geometry>
       </collision>
+      <xacro:default_inertial mass="0.001"/>
       <!-- <xacro:box_inertia m="0.1" w="0.1" d="0.1" h="0.1"/> -->
     </link>
-    <joint name="nav_gps_joint" type="fixed">
-      <parent link="base_link"/>
-      <child link="nav_gps_link"/>
-      <origin xyz="0 0 0.01"/>
-    </joint>
-    <gazebo reference="nav_gps_link">
-        <sensor name="nav_gps_sensor" type="gps">
-            <plugin name="nav_gps_plugin" filename="libgazebo_ros_gps_sensor.so">
+    <gazebo reference="gps_link">
+        <sensor name="gps_sensor" type="gps">
+            <plugin name="gps_plugin" filename="libgazebo_ros_gps_sensor.so">
                 <ros>
-                  <namespace>/demo</namespace>
-                    <remapping>~/out:=gps</remapping>
+                  <!-- <namespace>/demo</namespace> -->
+                  <remapping>~/out:=gps/fix</remapping>
                 </ros>
                 <frame_name>gps_link</frame_name>
@@ -245,13 +245,13 @@
               <longitude>
                   <mean>0.0</mean>
-                  <stddev>2e-4</stddev>
-                  <bias_mean>0.0000075</bias_mean>
-                  <bias_stddev>0.0000008</bias_stddev>
+                  <stddev>0.01</stddev>
+                  <!-- <bias_mean>0.0000075</bias_mean>
+                  <bias_stddev>0.0000008</bias_stddev> -->
               </longitude>
               <latitude>
                   <mean>0.0</mean>
-                  <stddev>2e-4</stddev>
-                  <bias_mean>0.0000075</bias_mean>
-                  <bias_stddev>0.0000008</bias_stddev>
+                  <stddev>0.01</stddev>
+                  <!-- <bias_mean>0.0000075</bias_mean>
+                  <bias_stddev>0.0000008</bias_stddev> -->
               </latitude>
             </gps>
@@ -259,4 +259,12 @@
         <material>Gazebo/Grey</material> <!-- TODO: fix? -->
     </gazebo>
+    <joint name="gps_joint" type="fixed">
+      <parent link="base_link"/>
+      <child link="gps_link"/>
+      <origin xyz="0 0 0.01"/>
+      <axis>
+          <xyz>0 0 1</xyz>
+        </axis>
+    </joint>
   </xacro:macro>
 </robot>

File: uwrt_mars_rover_drivetrain/uwrt_mars_rover_drivetrain_description/urdf/drivetrain.urdf.xacro (robot description, xacro)
@@ -37,4 +37,7 @@
     <origin xyz="0 0 ${wheel_diameter/2}" rpy="0 0 0"/>
   </joint>
+  <!-- sensors -->
+  <xacro:nav_imu/>
+  <xacro:nav_gps/>
   <!-- wheels -->
   <xacro:wheel prefix="right" suffix="front" parent_link="chassis" reflect="-1" x_position="${chassis_length/2}"/>
@@ -52,5 +55,3 @@
   <!-- <xacro:generate_sensor_frame sensor_params="${sensors_parameters['lidar']['lidar1']}"         name="lidar1"/>
   <xacro:default_lidar_frame lidar_link_name="lidar1" lidar_props="${sensors_parameters['lidar']['lidar1']['lidar_properties']}"/> -->
-  <xacro:nav_imu/>
-  <xacro:nav_gps/>
 </robot>

Commit message: fuse odometry data using robot localization

File: uwrt_mars_rover_drivetrain/uwrt_mars_rover_drivetrain_description/urdf/drivetrain.macro.xacro (robot description, xacro)
@@ -29,5 +29,5 @@
           iyy="1e-3" iyz="0.0"
           izz="1e-3"/>
-    </inertial>
+      </inertial>
   </xacro:macro>
    <xacro:macro name="chassis_inertia" params="chassis_width:=^ chassis_height:=^ chassis_length:=^ chassis_mass:=^">
@@ -117,3 +117,150 @@
     </ros2_control>
   </xacro:macro>
+  <xacro:macro name="nav_imu">
+    <link name="nav_imu_link">
+      <visual>
+        <geometry>
+          <box size="0.1 0.1 0.1"/>
+        </geometry>
+        <!-- <material name="cyan"> -->
+        <!--   <color rgba"0 1.0 1.0 1.0"/> -->
+        <!-- </material> -->
+      </visual>
+      <collision>
+        <geometry>
+          <box size="0.1 0.1 0.1"/>
+        </geometry>
+      </collision>
+      <xacro:default_inertial mass="0.001"/>
+    </link>
+    <gazebo reference="nav_imu_link">
+      <sensor name="nav_imu_sensor" type="imu">
+       <plugin filename="libgazebo_ros_imu_sensor.so" name="imu_plugin">
+          <ros>
+            <remapping>~/out:=imu/data</remapping>
+          </ros>
+          <initial_orientation_as_reference>false</initial_orientation_as_reference>
+        </plugin>
+        <always_on>true</always_on>
+        <update_rate>100</update_rate>
+        <visualize>true</visualize>
+        <imu>
+          <angular_velocity>
+            <x>
+              <noise type="gaussian">
+                <mean>0.0</mean>
+                <stddev>2e-4</stddev>
+                <!-- <bias_mean>0.0000075</bias_mean>
+                <bias_stddev>0.0000008</bias_stddev> -->
+              </noise>
+            </x>
+            <y>
+              <noise type="gaussian">
+                <mean>0.0</mean>
+                <stddev>2e-4</stddev>
+                <!-- <bias_mean>0.0000075</bias_mean>
+                <bias_stddev>0.0000008</bias_stddev> -->
+              </noise>
+            </y>
+            <z>
+              <noise type="gaussian">
+                <mean>0.0</mean>
+                <stddev>2e-4</stddev>
+                <!-- <bias_mean>0.0000075</bias_mean>
+                <bias_stddev>0.0000008</bias_stddev> -->
+              </noise>
+            </z>
+          </angular_velocity>
+          <linear_acceleration>
+            <x>
+              <noise type="gaussian">
+                <mean>0.0</mean>
+                <stddev>1.7e-2</stddev>
+                <!-- <bias_mean>0.1</bias_mean>
+                <bias_stddev>0.001</bias_stddev> -->
+              </noise>
+            </x>
+            <y>
+              <noise type="gaussian">
+                <mean>0.0</mean>
+                <stddev>1.7e-2</stddev>
+                <!-- <bias_mean>0.1</bias_mean>
+                <bias_stddev>0.001</bias_stddev> -->
+              </noise>
+            </y>
+            <z>
+              <noise type="gaussian">
+                <mean>0.0</mean>
+                <stddev>1.7e-2</stddev>
+                <!-- <bias_mean>0.1</bias_mean>
+                <bias_stddev>0.001</bias_stddev> -->
+              </noise>
+            </z>
+          </linear_acceleration>
+        </imu>
+      </sensor>
+    </gazebo>
+    <joint name="nav_imu_joint" type="fixed">
+      <parent link="base_link"/>
+      <child link="nav_imu_link"/>
+      <origin xyz ="0 0 0.1"/>
+      <axis>
+          <xyz>0 0 1</xyz>
+      </axis>
+    </joint>
+  </xacro:macro>
+  <xacro:macro name="nav_gps">
+    <link name="gps_link">
+      <visual>
+        <geometry>
+          <box size="0.1 0.1 0.1"/>
+        </geometry>
+        <!-- <material name="cyan"> -->
+        <!--   <color rgba"0 1.0 1.0 1.0"/> -->
+        <!-- </material> -->
+      </visual>
+      <collision>
+        <geometry>
+          <box size="0.1 0.1 0.1"/>
+        </geometry>
+      </collision>
+      <xacro:default_inertial mass="0.001"/>
+    </link>
+    <gazebo reference="gps_link">
+        <sensor name="gps_sensor" type="gps">
+            <plugin name="gps_plugin" filename="libgazebo_ros_gps_sensor.so">
+                <ros>
+                  <remapping>~/out:=gps/fix</remapping>
+                </ros>
+                <frame_name>gps_link</frame_name>
+            </plugin>
+            <always_on>true</always_on>
+            <update_rate>100</update_rate>
+            <visualize>true</visualize>
+            <gps>
+              <longitude>
+                  <mean>0.0</mean>
+                  <stddev>0.01</stddev>
+                  <!-- <bias_mean>0.0000075</bias_mean>
+                  <bias_stddev>0.0000008</bias_stddev> -->
+              </longitude>
+              <latitude>
+                  <mean>0.0</mean>
+                  <stddev>0.01</stddev>
+                  <!-- <bias_mean>0.0000075</bias_mean>
+                  <bias_stddev>0.0000008</bias_stddev> -->
+              </latitude>
+            </gps>
+        </sensor>
+        <material>Gazebo/Grey</material> <!-- TODO: fix? -->
+    </gazebo>
+    <joint name="gps_joint" type="fixed">
+      <parent link="base_link"/>
+      <child link="gps_link"/>
+      <origin xyz="0 0 0.1"/>
+      <axis>
+          <xyz>0 0 1</xyz>
+      </axis>
+    </joint>
+  </xacro:macro>
 </robot>

File: uwrt_mars_rover_drivetrain/uwrt_mars_rover_drivetrain_description/urdf/drivetrain.urdf.xacro (robot description, xacro)
@@ -37,4 +37,7 @@
     <origin xyz="0 0 ${wheel_diameter/2}" rpy="0 0 0"/>
   </joint>
+  <!-- sensors -->
+  <xacro:nav_imu/>
+  <xacro:nav_gps/>
   <!-- wheels -->
   <xacro:wheel prefix="right" suffix="front" parent_link="chassis" reflect="-1" x_position="${chassis_length/2}"/>
